File: kicad/ibm-modern-m-ssk.kicad_pcb (KiCad board)
At the start: 2 copper layers, 106 x 50 mm, 33 parts, among them J1 S2B-PH-SM4-TB(LF)(SN), J2 726386-2, J3 TF38-24S-0.5SV(830), J5 Conn_01x04_Pin, Q1 DMP2123LQ, Q2 DMP2123LQ, SW89 SW_Push, U1 MCP73831T-2DCI/MC, U2 TPS7A0233DQNR, U3 KESD0524P, U4 MDBT50Q-1MV2, Y1 32.768 kHz

Commit message: update mcu
Parts:
- removed D2: Blue, LED_SMD:LED_0201_0603Metric
- removed D3: B0530W, easyeda2kicad:SOD-123_L2.8-W1.8-LS3.7-RD
- removed D4: ESD5B5.0ST1G, easyeda2kicad:SOD-523_L1.2-W0.8-LS1.6-BI
- removed J3: TF38-24S-0.5SV(830), easyeda2kicad:FPC-SMD_24P-P0.50_TF38-24S-0.5SV-830
- removed Q2: DMP2123LQ, easyeda2kicad:SOT-23-3_L2.9-W1.3-P1.90-LS2.4-BR
- removed R10: 5.1k, Resistor_SMD:R_0402_1005Metric
- removed SW89: SW_Push, easyeda2kicad:SW-SMD_L3.9-W3.0-P4.45
- added C10: NC, Capacitor_SMD:C_0402_1005Metric, F.Cu at (98.8, 103.7)
- added C11: 100p, Capacitor_SMD:C_0402_1005Metric, F.Cu at (98.8, 105.7)
- added C12: 100n, Capacitor_SMD:C_0402_1005Metric, F.Cu at (98.8, 107.7)
- added C13: NC, Capacitor_SMD:C_0402_1005Metric, F.Cu at (98.8, 109.6)
- added C14: 1u, Capacitor_SMD:C_0603_1608Metric, F.Cu at (75.2, 106.5)
- added C15: 1u, Capacitor_SMD:C_0603_1608Metric, F.Cu at (75.2, 109.0)
- added C16: 47n, Capacitor_SMD:C_0402_1005Metric, F.Cu at (101.7, 103.7)
- added C17: 12p, Capacitor_SMD:C_0402_1005Metric, F.Cu at (101.7, 105.7)
- added C18: 12p, Capacitor_SMD:C_0402_1005Metric, F.Cu at (101.7, 107.7)
- added C19: 4.7u, Capacitor_SMD:C_0603_1608Metric, F.Cu at (75.2, 111.5)
- added C20: 4.7u, Capacitor_SMD:C_0603_1608Metric, F.Cu at (75.2, 114.0)
- added C21: 4.7u, Capacitor_SMD:C_0603_1608Metric, F.Cu at (79.2, 104.0)
- added C22: NC, Capacitor_SMD:C_0402_1005Metric, F.Cu at (101.7, 109.6)
- added C23: 4.7u, Capacitor_SMD:C_0603_1608Metric, F.Cu at (79.2, 106.5)
- added C24: 4.7u, Capacitor_SMD:C_0603_1608Metric, F.Cu at (79.2, 109.0)
- added C25: 4.7u, Capacitor_SMD:C_0603_1608Metric, F.Cu at (79.2, 111.5)
- added C26: 1u, Capacitor_SMD:C_0603_1608Metric, F.Cu at (79.2, 114.0)
- added C6: 4.7u, Capacitor_SMD:C_0603_1608Metric, F.Cu at (75.2, 104.0)
- added C7: 100n, Capacitor_SMD:C_0402_1005Metric, F.Cu at (96.0, 105.7)
- added C8: 100n, Capacitor_SMD:C_0402_1005Metric, F.Cu at (96.0, 107.7)
- added C9: 820p, Capacitor_SMD:C_0402_1005Metric, F.Cu at (96.0, 109.6)
- added E1: TPD2E001DRYR-TP, easyeda2kicad:SON-6_L1.4-W1.0-P0.50-TL_USBULC6-2M6, F.Cu at (74.5, 63.1)
- added J4: Conn_01x04_Pin, Connector_PinHeader_2.54mm:PinHeader_1x04_P2.54mm_Vertical, F.Cu at (52.5, 60.3)
- added L1: 4.7n, Inductor_SMD:L_0402_1005Metric, F.Cu at (80.0, 76.0)
- added L2: 10u, Inductor_SMD:L_0603_1608Metric_Pad1.05x0.95mm_HandSolder, F.Cu at (69.9, 117.8)
- added L3: 15n, Inductor_SMD:L_0402_1005Metric, F.Cu at (87.3, 105.7)
- added SW90: SW_Push, easyeda2kicad:SW-SMD_L3.9-W3.0-P4.45, F.Cu at (57.5, 56.0)
- added Y2: 32.768 kHz, Crystal:Crystal_SMD_3215-2Pin_3.2x1.5mm, F.Cu at (66.5, 75.5)
- C1: value 4.7u -> 12p; footprint Capacitor_SMD:C_0201_0603Metric -> Capacitor_SMD:C_0402_1005Metric
- C2: footprint Capacitor_SMD:C_0201_0603Metric -> Capacitor_SMD:C_0402_1005Metric
- C3: value 4.7u -> 0.8p; footprint Capacitor_SMD:C_0201_0603Metric -> Capacitor_SMD:C_0402_1005Metric
- C4: value 10u -> 0.5p; footprint Capacitor_SMD:C_0201_0603Metric -> Capacitor_SMD:C_0402_1005Metric
- C5: value 12p -> 100n; footprint Capacitor_SMD:C_0201_0603Metric -> Capacitor_SMD:C_0402_1005Metric
- J1: value S2B-PH-SM4-TB(LF)(SN) -> TF38-24S-0.5SV(830); footprint easyeda2kicad:CONN-SMD_2P-P1.00_SM02B-SRSS-TB-LF-SN -> easyeda2kicad:FPC-SMD_24P-P0.50_TF38-24S-0.5SV-830
- J2: value 726386-2 -> S2B-PH-SM4-TB(LF)(SN); footprint easyeda2kicad:CONN-TH_726386-2 -> easyeda2kicad:CONN-SMD_2P-P1.00_SM02B-SRSS-TB-LF-SN
- J5: value Conn_01x04_Pin -> 726386-2; footprint Connector_PinHeader_2.54mm:PinHeader_1x04_P2.54mm_Vertical -> easyeda2kicad:CONN-TH_726386-2
- R1: value 2k -> 1.5k
- R2: value 806k -> 4.7k
- R3: value 1k -> 4.7k
- R4: value 2M -> 10k
- R5: value 470 -> 47k
- R6: value 100k -> 1.8k
- R7: value 5.1k -> 10k
- R8, R9: value 27 -> 5.1k
- U1: value MCP73831T-2DCI/MC -> ~; footprint easyeda2kicad:DFN-8_L3.0-W2.0-P0.50-BL-EP1.6 -> nrf52840_qiaa:AQFN50P700X700X85_HS-74N
- U2: value TPS7A0233DQNR -> BQ24075RGTR; footprint easyeda2kicad:X2SON-4_L1.0-W1.0-P0.65-TL-EP -> easyeda2kicad:QFN-16_L3.0-W3.0-P0.50-TL-EP1.7
- U3: value KESD0524P -> XC6220B331ER-G; footprint easyeda2kicad:DFN2510-10_L2.5-W1.0-P0.50-BL -> easyeda2kicad:USP-6C_L2.0-W1.8-P0.50-BL-EP
- U4: value MDBT50Q-1MV2 -> LC709203FXE-03MH; footprint RF_Module:Raytac_MDBT50Q -> easyeda2kicad:WLCSP-9_L1.6-W1.8-R3-C3-P0.50-BL
- Y1: value 32.768 kHz -> 32MHz; footprint easyeda2kicad:FC-135R_L3.2-W1.5 -> Crystal:Crystal_SMD_2016-4Pin_2.0x1.6mm
- moved J5 83.8 mm to (54.5, 93.5), turned to 0 degrees
- moved C4 75.0 mm to (93.1, 109.6)
- moved C3 74.8 mm to (93.1, 107.7)
- moved C2 74.7 mm to (93.1, 105.7)
- moved C1 74.6 mm to (93.1, 103.7)
- moved C5 72.9 mm to (96.0, 103.7)
- moved R3 71.8 mm to (87.3, 111.7)
- moved R2 71.8 mm to (87.3, 109.7)
- moved R4 71.8 mm to (87.3, 113.7)
- moved R6 70.4 mm to (90.2, 105.7)
- moved R7 70.4 mm to (90.2, 107.7)
- moved R8 70.4 mm to (90.2, 109.7)
- moved R9 70.4 mm to (90.2, 111.7)
- moved R5 66.1 mm to (90.2, 103.7)
- moved J1 63.9 mm to (141.2, 53.4), turned to 0 degrees
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Connections:
- C1 pad 1: VBAT -> GND
- C1 pad 2: GND -> Net-(U1-XC1)
- C2 pad 2: Net-(U4-P0.00) -> Net-(U1-XC2)
- C3 pad 1: Net-(D3-K) -> Net-(U1-ANT)
- C4 pad 1: VDD_NRF -> Net-(C22-Pad1)
- C5 pad 1: Net-(U4-P0.01) -> GND
- C5 pad 2: GND -> Net-(U1-DEC1)
- D1 pad 2: VBUS -> SYS_PWR
- J1 pad 1: Net-(Q2-S) -> unconnected-(J1-Pad1)
- J1 pad 2: GND -> unconnected-(J1-Pad2)
- J1 pad 3: GND -> unconnected-(J1-Pad3)
- J1 pad 4: GND -> unconnected-(J1-Pad4)
- J2 pad 1: GND -> Net-(Q1-S)
- J5 pad 1: VDD_NRF -> GND
- Q1 pad 1: VBUS -> GND
- Q1 pad 2: Net-(D3-K) -> Net-(Q1-S)
- R1 pad 1: Net-(U1-PROG) -> Net-(D1-K)
- R1 pad 2: GND -> Net-(U2-#CHG)
- R2 pad 1: VBAT -> SCL
- R2 pad 2: BVOLT -> VDD_NRF
- R3 pad 1: STAT -> SDA
- R3 pad 2: Net-(D1-K) -> VDD_NRF
- R4 pad 1: BVOLT -> Net-(U4-TSENSE)
- R5 pad 2: Net-(D2-K) -> Net-(U2-TMR)
- R6 pad 2: VBUS -> Net-(U2-ISET)
- R7 pad 2: Net-(USBC1-CC1) -> Net-(U2-TS)
- R8 pad 1: D- -> GND
- R8 pad 2: Net-(U4-D-) -> Net-(USBC1-CC1)
- R9 pad 1: D+ -> GND
- R9 pad 2: Net-(U4-D+) -> Net-(USBC1-CC2)
- U2 pad 1: VDD_NRF -> Net-(U2-TS)
- U2 pad 2: GND -> VBAT
- U2 pad 3: Net-(D3-K) -> VBAT
- U2 pad 4: Net-(D3-K) -> GND
- U3 pad 1: ConnD+ -> VDD_NRF
- U3 pad 2: ConnD- -> VDD_NRF
- U3 pad 3: GND -> SYS_PWR
- U3 pad 4: unconnected-(U3-Pad4) -> GND
- U3 pad 5: unconnected-(U3-Pad5) -> SYS_PWR
- U3 pad 6: unconnected-(U3-Pad6) -> SYS_PWR
- U3 pad 7: unconnected-(U3-Pad7) -> GND
- USBC1 pad A4B9: VBUS -> ConnVBUS
- USBC1 pad B4A9: VBUS -> ConnVBUS
- Y1 pad 1: Net-(U4-P0.01) -> Net-(U1-XC2)
- Y1 pad 2: Net-(U4-P0.00) -> Net-(U1-XC1)
Other:
- board size 106 x 50 mm -> 100 x 50 mm

Commit message: update
Parts:
- removed C19, C23, C24, C25: 4.7u, Capacitor_SMD:C_0603_1608Metric
- removed C26: 1u, Capacitor_SMD:C_0603_1608Metric
- removed D1: Red, LED_SMD:LED_0201_0603Metric
- removed R2, R3: 4.7k, Resistor_SMD:R_0402_1005Metric
- removed R4, R7: 10k, Resistor_SMD:R_0402_1005Metric
- removed R5: 47k, Resistor_SMD:R_0402_1005Metric
- removed R6: 1.8k, Resistor_SMD:R_0402_1005Metric
- removed U3: XC6220B331ER-G, easyeda2kicad:USP-6C_L2.0-W1.8-P0.50-BL-EP
- removed U4: LC709203FXE-03MH, easyeda2kicad:WLCSP-9_L1.6-W1.8-R3-C3-P0.50-BL
- added C27: 1u, Capacitor_SMD:C_0603_1608Metric, F.Cu at (127.5, 81.8)
- added C28: 2.2u, Capacitor_SMD:C_0603_1608Metric, F.Cu at (127.5, 84.3)
- added C29: 10u, Capacitor_SMD:C_0603_1608Metric, F.Cu at (127.5, 86.8)
- added C30: 10u, Capacitor_SMD:C_0603_1608Metric, F.Cu at (131.6, 79.3)
- added C31: 10u, Capacitor_SMD:C_0603_1608Metric, F.Cu at (131.6, 81.8)
- added C32: 1u, Capacitor_SMD:C_0603_1608Metric, F.Cu at (131.6, 84.3)
- added C33: 1u, Capacitor_SMD:C_0603_1608Metric, F.Cu at (131.6, 86.8)
- added D2: LED_RGB, easyeda2kicad:LED-SMD_4P-L1.6-W1.5-TR-1, F.Cu at (99.4, 80.2)
- added L4: 2.2u, Inductor_SMD:L_1008_2520Metric, F.Cu at (129.1, 93.2)
- added R10: 470k, Resistor_SMD:R_0402_1005Metric, F.Cu at (135.0, 89.0)
- R1: value 1.5k -> 10k
- U1: value ~ -> NRF52840
- U2: value BQ24075RGTR -> nPM1300-QEAA; footprint easyeda2kicad:QFN-16_L3.0-W3.0-P0.50-TL-EP1.7 -> Nordic_QFN50P500X500X90-33N:Nordic_QFN50P500X500X90-33N
- moved J4 69.7 mm to (119.2, 80.3), turned to 0 degrees
- moved J1 69.4 mm to (82.2, 89.8)
- moved BT1 63.0 mm to (191.5, 78.5)
- moved Y2 60.2 mm to (124.1, 93.0), turned to 0 degrees
- moved E1 59.7 mm to (134.0, 57.9)
- moved R1 59.7 mm to (135.0, 83.0), turned to 0 degrees
- moved SW90 56.3 mm to (108.3, 80.3), turned to 0 degrees
- moved C20 55.5 mm to (123.5, 86.8)
- moved L1 55.1 mm to (135.0, 79.0)
- moved C14 54.3 mm to (123.5, 81.8)
- moved C15 54.3 mm to (123.5, 84.3)
- moved C6 54.3 mm to (123.5, 79.3)
- moved C21 54.3 mm to (127.5, 79.3)
- moved L3 53.8 mm to (135.0, 81.0)
- moved J2 51.3 mm to (63.0, 88.5), turned to 0 degrees
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Connections:
- C21 pad 1: ConnVBUS -> VBUSOUT
- R1 pad 1: Net-(D1-K) -> GND
- R1 pad 2: Net-(U2-#CHG) -> Net-(JP1-A)
- R8 pad 2: Net-(USBC1-CC1) -> CC1
- R9 pad 2: Net-(USBC1-CC2) -> CC2
- U1 pad AD2: ConnVBUS -> VBUSOUT
- U2 pad 1: Net-(U2-TS) -> VSYS
- U2 pad 10: SYS_PWR -> unconnected-(U2-GPIO3-Pad10)
- U2 pad 11: SYS_PWR -> unconnected-(U2-GPIO4-Pad11)
- U2 pad 12: unconnected-(U2-ILIM-Pad12) -> VDD_NRF
- U2 pad 13: ConnVBUS -> SDA
- U2 pad 14: Net-(U2-TMR) -> SCL
- U2 pad 15: GND -> unconnected-(U2-SHPHLD-Pad15)
- U2 pad 2: VBAT -> GND
- U2 pad 3: VBAT -> unconnected-(U2-SW1-Pad3)
- U2 pad 4: GND -> VSYS
- U2 pad 5: GND -> Net-(U2-SW2)
- U2 pad 6: ConnVBUS -> GND
- U2 pad 8: GND -> unconnected-(U2-GPIO1-Pad8)
- U2 pad 9: Net-(U2-#CHG) -> unconnected-(U2-GPIO2-Pad9)
- USBC1 pad A5: Net-(USBC1-CC1) -> CC1
- USBC1 pad B5: Net-(USBC1-CC2) -> CC2

Commit message: update - pcb layout
Parts:
- moved J2 96.3 mm to (149.8, 46.8)
- moved C17 93.3 mm to (53.5, 74.0), turned to 90 degrees
- moved C18 90.8 mm to (56.0, 75.8)
- moved C16 86.9 mm to (60.0, 70.5)
- moved C5 84.3 mm to (56.8, 72.2)
- moved C12 79.4 mm to (65.2, 70.5)
- moved C7 78.0 mm to (62.8, 80.0), turned to -90 degrees
- moved L3 76.7 mm to (59.5, 67.8), turned to 180 degrees
- moved C11 76.3 mm to (68.0, 71.0), turned to 180 degrees
- moved C10 75.7 mm to (68.2, 72.5), turned to 90 degrees
- moved C8 75.3 mm to (65.5, 80.0), turned to -90 degrees
- moved C2 74.0 mm to (65.0, 68.5), turned to -90 degrees
- moved C9 73.2 mm to (68.0, 76.8), turned to 180 degrees
- moved J1 73.0 mm to (134.5, 38.9)
- moved C3 71.5 mm to (67.0, 73.8), turned to 90 degrees
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Other:
- copper layers 2 -> 4

Commit message: update
Parts:
- added J6: Conn_Coaxial_Small, easyeda2kicad:IPEX-SMD_3P-L2.6-W2.6-LS3.0_ZCF-CF0001-0002IPEX, F.Cu at (53.9, 86.0)
- added JP1: SolderJumper_2_Open, Jumper:SolderJumper-2_P1.3mm_Open_RoundedPad1.0x1.5mm, F.Cu at (186.0, 27.5)
- Q1: value DMP2123LQ -> PMZB350UPE,315; footprint easyeda2kicad:SOT-23-3_L2.9-W1.3-P1.90-LS2.4-BR -> Package_DFN_QFN:Diodes_DFN1006-3
- moved R1 101.4 mm to (181.5, 27.2)
- moved Q1 85.3 mm to (184.6, 22.0)
- moved D2 60.5 mm to (107.7, 20.2)
- moved E1 50.0 mm to (102.2, 19.2)
- moved R9 46.4 mm to (110.2, 29.7)
- moved R8 46.4 mm to (110.2, 27.8)
- moved C22 46.3 mm to (158.5, 44.7)
- moved C13 46.3 mm to (158.1, 40.9)
- moved L4 44.9 mm to (84.2, 90.0), turned to -90 degrees
- moved SW90 39.9 mm to (116.5, 41.2)
- moved J2 33.8 mm to (174.5, 23.8)
- moved J1 29.8 mm to (108.2, 53.0)
- moved C31 29.3 mm to (96.5, 92.0)
- moved L2 27.1 mm to (70.0, 92.5), turned to 90 degrees
- moved L3 26.9 mm to (68.0, 93.2), turned to 0 degrees
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- renumbered Y1 to Yr1
Connections:
- J2 pad 1: Net-(Q1-S) -> Net-(J2-Pad1)
- Q1 pad 1: GND -> (no net)
- Q1 pad 2: Net-(Q1-S) -> (no net)
- Q1 pad 3: VBAT -> (no net)
- Y2 pad 1: Net-(U1-P0.00/XL1) -> Net-(U1-P0.01/XL2)
- Y2 pad 2: Net-(U1-P0.01/XL2) -> Net-(U1-P0.00/XL1)
- Yr1 pad 2: Net-(U1-XC1) -> GND
- Yr1 pad 3: (no net) -> Net-(U1-XC1)
- Yr1 pad 4: (no net) -> GND
Routing:
- net VDD_NRF: track 0.00 -> 10.1 mm
- net Net-(U1-DEC4): track 0.00 -> 8.42 mm
- net Net-(U1-P0.00/XL1): track 0.00 -> 6.91 mm
- net Net-(U1-XC1): track 0.00 -> 5.98 mm
- net Net-(U1-XC2): track 0.00 -> 5.11 mm
- net Net-(U1-P0.01/XL2): track 0.00 -> 4.84 mm
- net Net-(U1-DCC): track 0.00 -> 3.87 mm
- net Net-(U1-DECUSB): track 0.00 -> 3.16 mm
- net Net-(U1-DEC3): track 0.00 -> 3.07 mm
- net Net-(U1-DEC5): track 0.00 -> 2.92 mm
- net Net-(U1-ANT): track 0.00 -> 2.92 mm
- net Net-(U1-DEC1): track 0.00 -> 2.86 mm
- net VBUSOUT: track 0.00 -> 1.87 mm
- net Net-(L2-Pad1): track 0.00 -> 1.55 mm
- net Net-(J6-In): track 0.00 -> 1.02 mm
