File: kicad/ibm-modern-m-ssk.kicad_pcb (KiCad board)
At the start: 4 copper layers, 100 x 50 mm, 52 parts, among them J1 TF38-24S-0.5SV(830), J2 S2B-PH-SM4-TB(LF)(SN), J4 Conn_01x04_Pin, J5 726386-2, J6 Conn_Coaxial_Small, Q1 PMZB350UPE,315, SW90 SW_Push, U1 NRF52840, U2 nPM1300-QEAA, Y2 32.768 kHz

Commit message: update
Parts:
- removed JP1: SolderJumper_2_Open, Jumper:SolderJumper-2_P1.3mm_Open_RoundedPad1.0x1.5mm
- BT1: value Li-Po 603450 -> LP803040; footprint easyeda2kicad:LiPo_603450 -> easyeda2kicad:LP803040
- J2: value S2B-PH-SM4-TB(LF)(SN) -> Molex PicoBlade; footprint easyeda2kicad:CONN-SMD_2P-P1.00_SM02B-SRSS-TB-LF-SN -> Connector_Molex:Molex_PicoBlade_53261-0271_1x02-1MP_P1.25mm_Horizontal
- moved C13 103.1 mm to (234.1, 110.5)
- moved C22 103.1 mm to (234.5, 114.4)
- moved Q1 89.5 mm to (132.6, 94.8), turned to 180 degrees
- moved J2 78.1 mm to (142.0, 94.8), turned to -90 degrees
- moved BT1 67.4 mm to (124.3, 73.7)
- moved SW90 54.8 mm to (106.4, 95.1)
- moved USBC1 48.2 mm to (124.3, 72.7)
- moved D2 47.8 mm to (75.0, 55.0)
- moved R1 46.2 mm to (136.1, 35.9)
- moved J4 41.3 mm to (82.0, 98.1), turned to 90 degrees
- moved C27 4.86 mm to (94.2, 86.2)
- moved C28 4.86 mm to (94.2, 89.5)
- moved C29 4.86 mm to (85.0, 83.0)
- moved C30 4.86 mm to (84.2, 85.2)
- moved C31 4.86 mm to (94.2, 87.7)
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Connections:
- J2 pad 1: Net-(J2-Pad1) -> Net-(Q1-S)
- Q1 pad 1: (no net) -> GND
- Q1 pad 2: (no net) -> Net-(Q1-S)
- Q1 pad 3: (no net) -> VBAT
- R1 pad 2: Net-(JP1-A) -> Net-(U2-NTC)
- U2 pad 18: Net-(JP1-B) -> Net-(U2-NTC)

Commit message: update
Parts:
- removed E1: TPD2E001DRYR-TP, easyeda2kicad:SON-6_L1.4-W1.0-P0.50-TL_USBULC6-2M6
- added D1: PESDNC2FD5VB, easyeda2kicad:Diodes_DFN1006-2, F.Cu at (190.2, 50.4)
- added F1: BSMD0603L-150, Fuse:Fuse_0603_1608Metric, F.Cu at (188.4, 49.7)
- added U3: TPD4E05U06DQAR, Package_SON:USON-10_2.5x1.0mm_P0.5mm, F.Cu at (195.0, 50.1)
- moved BT1 137.5 mm to (258.8, 45.4)
- moved J1 75.6 mm to (195.0, 46.0), turned to 180 degrees
- renumbered USBC1 to J1, J1 to J7
Connections:
- net ConnD+ renamed D+
- net ConnD- renamed D-
- net ConnVBUS renamed VBUS
- R8 pad 1: GND -> unconnected-(R8-Pad1)
- R8 pad 2: CC1 -> unconnected-(R8-Pad2)
- R9 pad 1: GND -> unconnected-(R9-Pad1)
- R9 pad 2: CC2 -> unconnected-(R9-Pad2)
Routing:
- net VBUS: track 0.00 -> 13.3 mm, vias 0 -> 3
- net VDD_NRF: track 10.1 -> 0.00 mm
- net Net-(U1-DEC4): track 8.43 -> 0.00 mm
- net D+: track 0.00 -> 8.23 mm, vias 0 -> 2
- net D-: track 0.00 -> 7.11 mm, vias 0 -> 2
- net Net-(U1-P0.00/XL1): track 6.92 -> 0.00 mm
- net Net-(U1-XC1): track 5.98 -> 0.00 mm
- net Net-(U1-XC2): track 5.11 -> 0.00 mm
- net Net-(U1-P0.01/XL2): track 4.84 -> 0.00 mm
- net Net-(U1-DCC): track 3.87 -> 0.00 mm
- net Net-(U1-DECUSB): track 3.16 -> 0.00 mm
- net Net-(U1-DEC3): track 3.07 -> 0.00 mm
- net Net-(U1-DEC5): track 2.92 -> 0.00 mm
- net Net-(U1-ANT): track 2.92 -> 0.00 mm
- net Net-(U1-DEC1): track 2.86 -> 0.00 mm
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Other:
- board size 100 x 50 mm -> 154.1 x 57.4 mm

Commit message: update
Parts:
- removed D2: LED_RGB, easyeda2kicad:LED-SMD_4P-L1.6-W1.5-TR-1
- removed R1: 10k, Resistor_SMD:R_0402_1005Metric
- removed R8, R9: 5.1k, Resistor_SMD:R_0402_1005Metric
- added D4: rgb, LED_SMD:LED_Wurth_150044M155260, F.Cu at (118.3, 83.0)
- added D92: rgb, LED_SMD:LED_Wurth_150044M155260, F.Cu at (129.6, 82.9)
- added J8: FPC_12P_0.5mm, easyeda2kicad:FPC_12P_0.5mm, F.Cu at (123.8, 78.2)
- added J9: FH12-12S-0.5SVA(54), easyeda2kicad:FH1212S05SVA54, F.Cu at (75.1, 67.4)
- added REF**: MouseBite-Slot_2.0x2.0mm_outset_D0.5mm_P0.85mm_3h, Panelization:MouseBite-Slot_2.0x2.0mm_outset_D0.5mm_P0.85mm_3h, F.Cu at (114.2, 82.9)
- added REF**: MouseBite-Slot_2.0x2.0mm_outset_D0.5mm_P0.85mm_3h, Panelization:MouseBite-Slot_2.0x2.0mm_outset_D0.5mm_P0.85mm_3h, F.Cu at (133.5, 82.9)
- added REF**: db_holder, easyeda2kicad:db_holder, F.Cu at (75.0, 56.0)
- added SW89: SW_Push, easyeda2kicad:SW-SMD_2P-L3.0-W2.5-LS4.0, F.Cu at (115.7, 82.9)
- added SW91: SW_Push, easyeda2kicad:SW-SMD_2P-L3.0-W2.5-LS4.0, F.Cu at (132.0, 82.9)
- J1: value TYPE-C-31-M-12 -> TYPE-C-31-D-06; footprint easyeda2kicad:USB-C_SMD-TYPE-C-31-M-12_1 -> easyeda2kicad:USB-C-SMD_TYPE-C-31-D-06
- moved C13 162.3 mm to (72.4, 124.2)
- moved C22 162.3 mm to (72.8, 128.0)
- moved J1 80.2 mm to (123.8, 82.9), turned to 0 degrees
- moved U3 77.1 mm to (123.8, 79.9)
- moved D1 77.1 mm to (118.3, 78.4), turned to 0 degrees
- moved F1 76.3 mm to (118.3, 79.9), turned to 180 degrees
- moved C27 5.49 mm to (89.8, 83.0)
- moved C31 5.49 mm to (89.8, 84.5)
- moved R10 5.39 mm to (86.7, 87.8)
- moved C33 5.35 mm to (84.5, 79.6)
- moved C28 5.35 mm to (89.8, 86.5)
- moved C30 5.35 mm to (79.8, 82.3)
- moved C32 5.35 mm to (89.8, 80.8)
- moved L4 5.35 mm to (77.5, 82.8)
- moved U2 5.35 mm to (84.3, 83.8)
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Connections:
- C29 pad 2: GND -> PVSS1
- C30 pad 2: GND -> PVSS1
- D1 pad 2: VCOM -> VBUS
- F1 pad 1: VBUS -> Net-(F1-Pad1)
- F1 pad 2: VCOM -> VBUS
- L4 pad 2: Net-(U2-SW2) -> Net-(U2-SW1)
- Q1 pad 1: GND -> (no net)
- Q1 pad 2: Net-(Q1-S) -> (no net)
- Q1 pad 3: VBAT -> (no net)
- R10 pad 1: Net-(U2-VSET2) -> Net-(U2-VSET1)
- U2 pad 1: VSYS -> VDD_NRF
- U2 pad 12: VDD_NRF -> unconnected-(U2-VDDIO-Pad12)
- U2 pad 15: unconnected-(U2-SHPHLD-Pad15) -> SHPHLD
- U2 pad 16: Net-(U2-VSET2) -> GND
- U2 pad 17: GND -> Net-(U2-VSET1)
- U2 pad 2: GND -> PVSS1
- U2 pad 25: Net-(D2-RK) -> unconnected-(U2-LED0-Pad25)
- U2 pad 26: Net-(D2-GK) -> unconnected-(U2-LED1-Pad26)
- U2 pad 27: Net-(D2-BK) -> unconnected-(U2-LED2-Pad27)
- U2 pad 3: unconnected-(U2-SW1-Pad3) -> Net-(U2-SW1)
- U2 pad 32: VDD_NRF -> VSYS
- U2 pad 5: Net-(U2-SW2) -> unconnected-(U2-SW2-Pad5)
- U3 pad 2: D- -> D+
- U3 pad 4: D+ -> D-
- U3 pad 7: D+ -> D-
- U3 pad 9: D- -> D+
- Yr1 pad 4: GND -> unconnected-(Yr1-Pad4)
Routing:
- net VDD_NRF: track 0.00 -> 45.9 mm, vias 0 -> 7
- net GND: track 0.00 -> 43.7 mm, vias 0 -> 44
- net Net-(U1-DEC4): track 0.00 -> 20.7 mm, vias 0 -> 2
- net Net-(F1-Pad1): track 0.00 -> 16.4 mm, vias 0 -> 4
- net SHPHLD: track 0.00 -> 10.3 mm, vias 0 -> 3
- net BT_PAIR: track 0.00 -> 9.85 mm, vias 0 -> 2
- net CC2: track 2.62 -> 10.6 mm, vias 0 -> 3
- net Net-(U1-P0.00/XL1): track 0.00 -> 7.14 mm
- net VBUS: track 13.3 -> 6.61 mm, vias 3 -> 0
- net Net-(U1-XC1): track 0.00 -> 6.18 mm
- net CC1: track 2.17 -> 8.22 mm, vias 0 -> 1
- net D-: track 7.11 -> 12.8 mm
- net Net-(U1-P0.01/XL2): track 0.00 -> 5.34 mm
- net Net-(U2-SW1): track 0.00 -> 5.26 mm
- net Net-(U1-XC2): track 0.00 -> 5.13 mm
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- added copper zone on F.Cu, net GND
- added copper zone on F.Cu, net PVSS1
- added copper zone on F.Cu, net VBAT
- added copper zone on F.Cu, net VBUS
- added copper zone on F.Cu, net VDD_NRF
- added copper zone on B.Cu, net VSYS
- added copper zone on F.Cu, net VSYS
Other:
- board size 154.1 x 57.4 mm -> 100 x 50 mm

Commit message: update
Parts:
- removed the REF** at (75.0, 56.0)
- removed Yr1: 32MHz, Crystal:Crystal_SMD_2016-4Pin_2.0x1.6mm
- added Y1: 32MHz, Crystal:Crystal_SMD_2016-4Pin_2.0x1.6mm, F.Cu at (65.3, 83.5)
- SW90: footprint easyeda2kicad:SW-SMD_L3.9-W3.0-P4.45 -> easyeda2kicad:SW-SMD_2P-L3.0-W2.5-LS4.0
- moved BT1 157.1 mm to (121.8, 122.3)
- moved J2 48.4 mm to (112.8, 56.2), turned to 0 degrees
- moved REF** 34.1 mm to (102.1, 69.4), turned to 0 degrees
- moved SW91 32.2 mm to (102.2, 70.8), turned to 180 degrees
- moved D92 29.1 mm to (102.2, 73.3), turned to 90 degrees
- moved J8 26.5 mm to (97.4, 79.0), turned to 90 degrees
- moved U3 24.7 mm to (99.2, 79.0), turned to 180 degrees
- moved J1 22.0 mm to (102.2, 79.0), turned to 90 degrees
- moved D1 21.6 mm to (97.7, 84.5), turned to 90 degrees
- moved SW90 21.1 mm to (86.8, 87.5), turned to 90 degrees
- moved C17 19.7 mm to (59.3, 70.2), turned to 180 degrees
- moved F1 19.7 mm to (99.2, 84.5), turned to -90 degrees
- moved C6 16.6 mm to (53.8, 74.3), turned to 180 degrees
- moved C18 16.5 mm to (57.5, 72.8), turned to -90 degrees
- moved C32 16.5 mm to (74.8, 73.7), turned to 90 degrees
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Connections:
- net BT_PAIR renamed /daughterboard/BT_PAIR
- net CC1 renamed /daughterboard/CC1
- net CC2 renamed /daughterboard/CC2
- net LED_DATA renamed /daughterboard/LED_DATA
- net Net-(J6-In) renamed /motherboard/ANTENNA
- net Net-(U1-DEC4) renamed /motherboard/DEC4
- net RESET renamed /motherboard/RESET
- net SCL renamed /motherboard/SCL
- net SDA renamed /motherboard/SDA
- net SHPHLD renamed /daughterboard/SHPHLD
- C9 pad 1: GND -> Net-(U1-DEC5)
- C9 pad 2: Net-(U1-DEC5) -> GND
- J4 pad 2: SWCLK -> /motherboard/SWDIO
- J4 pad 3: SWDIO -> /motherboard/SWCLK
- Q1 pad 1: (no net) -> GND
- Q1 pad 2: (no net) -> Net-(Q1-S)
- Q1 pad 3: (no net) -> VBAT
- U1 pad AA24: SWCLK -> /motherboard/SWCLK
- U1 pad AC24: SWDIO -> /motherboard/SWDIO
Routing:
- net unconnected-(Yr1-Pad4): track 1.00 -> 0.00 mm, vias 1 -> 0
- net Net-(U1-DEC5): track 1.98 -> 2.73 mm, vias 0 -> 1
Other:
- outline, holes or cut-outs redrawn

Commit message: update
Parts:
- moved Q1 49.2 mm to (109.2, 51.5)
Changed lines of the file:
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@@
 	(footprint "Package_DFN_QFN:Diodes_DFN1006-3"
 		(layer "F.Cu")
-		(at 132.59999 94.8 180)
+		(at 109.25 51.5 180)
 		(descr "DFN package size 1006 3 pins")
 		(tags "DFN package size 1006 3 pins")

Commit message: update
Parts:
- removed J4: Conn_01x04_Pin, Connector_PinHeader_2.54mm:PinHeader_1x04_P2.54mm_Vertical
- added J10: TC2030, Connector:Tag-Connect_TC2030-IDC-NL_2x03_P1.27mm_Vertical, F.Cu at (71.3, 82.1)
- moved J6 20.7 mm to (60.0, 69.7), turned to 0 degrees
- moved C17 19.7 mm to (59.6, 89.9), turned to 0 degrees
- moved SW90 19.4 mm to (67.9, 92.1), turned to 0 degrees
- moved L2 16.6 mm to (53.5, 85.9), turned to 0 degrees
- moved C6 16.1 mm to (65.0, 85.9), turned to 0 degrees
- moved C1 15.8 mm to (53.5, 74.9), turned to 180 degrees
- moved L3 15.6 mm to (52.6, 83.9), turned to -90 degrees
- moved C18 15.1 mm to (61.4, 87.4), turned to 90 degrees
- moved C20 14.9 mm to (65.5, 84.4), turned to 0 degrees
- moved C14 14.8 mm to (56.0, 86.6), turned to 90 degrees
- moved Y2 14.6 mm to (59.6, 87.4), turned to 90 degrees
- moved Y1 13.7 mm to (53.5, 76.6), turned to -90 degrees
- moved C5 13.7 mm to (57.4, 86.6), turned to 90 degrees
- moved C4 13.5 mm to (58.5, 73.4), turned to 180 degrees
- moved C21 13.4 mm to (65.5, 82.9), turned to 0 degrees
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Other:
- board size 100 x 50 mm -> 75 x 50 mm

Commit message: update
Parts:
- removed BT1: LP803040, easyeda2kicad:LP803040
- removed C13, C22: NC, Capacitor_SMD:C_0402_1005Metric
- added J4: AFB10-S18LCA-00, easyeda2kicad:FPC-SMD_18P-P1.00_AFB10-S18LCA-00, F.Cu at (106.8, 67.7)
- D4, D92: footprint LED_SMD:LED_Wurth_150044M155260 -> easyeda2kicad:WS2812C-2020-V1
- J7: value TF38-24S-0.5SV(830) -> AFB10-S06LCA-00; footprint easyeda2kicad:FPC-SMD_24P-P0.50_TF38-24S-0.5SV-830 -> easyeda2kicad:FPC-SMD_6P-P1.00_AFB10-S6LCA-00
- J9: value FH12-12S-0.5SVA(54) -> AFC11-S12ICA-00; footprint easyeda2kicad:FH1212S05SVA54 -> easyeda2kicad:CONN-SMD-12P_AFC11-S12ICA-00
- Q1: footprint Package_DFN_QFN:Diodes_DFN1006-3 -> easyeda2kicad:DFN1006-3
- SW89, SW90, SW91: footprint easyeda2kicad:SW-SMD_2P-L3.0-W2.5-LS4.0 -> easyeda2kicad:KEY-SMD_B3U-1000PM
- Y1: footprint Crystal:Crystal_SMD_2016-4Pin_2.0x1.6mm -> easyeda2kicad:Crystal_SMD_2016-4Pin_2.0x1.6mm
- Y2: footprint Crystal:Crystal_SMD_3215-2Pin_3.2x1.5mm -> easyeda2kicad:Crystal_SMD_3215-2Pin
- moved Q1 57.9 mm to (101.6, 108.9)
- moved J2 49.5 mm to (110.8, 105.7), turned to 90 degrees
- moved J10 28.1 mm to (53.8, 104.1), turned to 180 degrees
- moved SW90 27.3 mm to (88.0, 110.7)
- moved J9 15.9 mm to (66.4, 79.7)
- moved J5 14.6 mm to (48.4, 110.7)
- moved J7 14.3 mm to (91.2, 67.7)
- moved D4 12.4 mm to (100.0, 96.7), turned to 180 degrees
- moved D1 12.3 mm to (95.4, 96.6)
- moved F1 12.3 mm to (96.9, 96.6)
- moved J1 12.3 mm to (99.9, 91.1)
- moved J8 12.3 mm to (95.2, 91.1)
- moved REF** 12.3 mm to (99.9, 100.7)
- moved REF** 12.3 mm to (99.9, 81.5)
- moved SW91 12.3 mm to (99.9, 82.9), turned to 0 degrees
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Routing:
- net GND: track 43.9 -> 43.4 mm, vias 44 -> 35
- removed copper zone on F.Cu, net GND
Other:
- outline, holes or cut-outs redrawn
