File: kicad/ibm-modern-m-ssk.kicad_sch (KiCad schematic)
At the start: 47 parts, among them J1 S2B-PH-SM4-TB(LF)(SN), J2 726386-2, J3 TF38-24S-0.5SV(830), J4 Conn_02x06_Odd_Even, J5 Conn_01x04_Pin, Q1 DMP2123LQ, Q2 DMP2123LQ, SW89 SW_Push, SW90 SW_SPDT, U1 MCP73831T-2DCI/MC, U2 TPS7A0233DQNR, U3 KESD0524P, U4 MDBT50Q-1MV2, U5 XC6220B331ER-G, U6 BQ24075RGTR, U7 LC709203FXE-03MH, Y1 32.768 kHz

Commit message: update mcu
Parts:
- removed D3: B0530W, easyeda2kicad:SOD-123_L2.8-W1.8-LS3.7-RD, symbol Device:D_Schottky_Small
- removed D4: ESD5B5.0ST1G, easyeda2kicad:SOD-523_L1.2-W0.8-LS1.6-BI, symbol easyeda2kicad:ESD5B5.0ST1G
- removed E1: PESD5V0S1BL,315, easyeda2kicad:SOD-882_L1.0-W0.6-BI, symbol Device:D_TVS_Small
- removed Q1: DMP2123LQ, easyeda2kicad:SOT-23-3_L2.9-W1.3-P1.90-LS2.4-BR, symbol easyeda2kicad:DMP2123LQ
- removed R1: 2k, Resistor_SMD:R_0402_1005Metric, symbol Device:R_Small
- removed R6: 100k, Resistor_SMD:R_0402_1005Metric, symbol Device:R_Small
- removed R8, R9: 27, Resistor_SMD:R_0402_1005Metric, symbol Device:R_Small
- removed SW90: SW_SPDT, symbol Switch:SW_SPDT
- removed U1: MCP73831T-2DCI/MC, easyeda2kicad:DFN-8_L3.0-W2.0-P0.50-BL-EP1.6, symbol easyeda2kicad:MCP73831T-2DCI_MC
- removed U2: TPS7A0233DQNR, easyeda2kicad:X2SON-4_L1.0-W1.0-P0.65-TL-EP, symbol easyeda2kicad:TPS7A0233DQNR
- removed U3: KESD0524P, easyeda2kicad:DFN2510-10_L2.5-W1.0-P0.50-BL, symbol easyeda2kicad:KESD0524P
- removed U4: MDBT50Q-1MV2, RF_Module:Raytac_MDBT50Q, symbol RF_Module:MDBT50Q-1MV2
- added C11: 100p, Capacitor_SMD:C_0402_1005Metric, symbol Device:C_Small
- added C12: 100n, Capacitor_SMD:C_0402_1005Metric, symbol Device:C_Small
- added C13, C22: NC, Capacitor_SMD:C_0402_1005Metric, symbol Device:C_Small
- added C14, C15, C26: 1u, Capacitor_SMD:C_0603_1608Metric, symbol Device:C_Small
- added C16: 47n, Capacitor_SMD:C_0402_1005Metric, symbol Device:C_Small
- added C17, C18: 12p, Capacitor_SMD:C_0402_1005Metric, symbol Device:C_Small
- added C19, C20, C21, C23, C24, C25: 4.7u, Capacitor_SMD:C_0603_1608Metric, symbol Device:C_Small
- added L1: 4.7n, Inductor_SMD:L_0402_1005Metric, symbol Device:L_Small
- added L2: 10u, Inductor_SMD:L_0603_1608Metric_Pad1.05x0.95mm_HandSolder, symbol Device:L_Small
- added L3: 15n, Inductor_SMD:L_0402_1005Metric, symbol Device:L_Small
- added U1: ~, nrf52840_qiaa:AQFN50P700X700X85_HS-74N, symbol nrf52840_qiaa_config5:root_0_nRF52840_QIAA_AltiumLib.DbLib
- added Y2: 32.768 kHz, Crystal:Crystal_SMD_3215-2Pin_3.2x1.5mm, symbol Device:Crystal_Small
- C1: value 4.7u -> 12p; footprint Capacitor_SMD:C_0201_0603Metric -> Capacitor_SMD:C_0402_1005Metric; LCSC Part C19666 -> C526985
- C10: value 10u -> NC; footprint Capacitor_SMD:C_0201_0603Metric -> Capacitor_SMD:C_0402_1005Metric; LCSC Part C19666 -> (none)
- C2: footprint Capacitor_SMD:C_0201_0603Metric -> Capacitor_SMD:C_0402_1005Metric; LCSC Part C38523 -> C526985
- C3: value 4.7u -> 0.8p; footprint Capacitor_SMD:C_0201_0603Metric -> Capacitor_SMD:C_0402_1005Metric; LCSC Part C19666 -> C326068
- C4: value 10u -> 0.5p; footprint Capacitor_SMD:C_0201_0603Metric -> Capacitor_SMD:C_0402_1005Metric; LCSC Part C1634 -> C327230
- C5: value 12p -> 100n; footprint Capacitor_SMD:C_0201_0603Metric -> Capacitor_SMD:C_0402_1005Metric; LCSC Part C38523 -> C60474
- C6: value 1u -> 4.7u; footprint Capacitor_SMD:C_0201_0603Metric -> Capacitor_SMD:C_0603_1608Metric; LCSC Part C19666 -> C277476
- C7: value 4.7u -> 100n; footprint Capacitor_SMD:C_0201_0603Metric -> Capacitor_SMD:C_0402_1005Metric; LCSC Part C19666 -> C60474
- C8: value 1u -> 100n; footprint Capacitor_SMD:C_0201_0603Metric -> Capacitor_SMD:C_0402_1005Metric; LCSC Part C19666 -> C60474
- C9: value 10u -> 820p; footprint Capacitor_SMD:C_0201_0603Metric -> Capacitor_SMD:C_0402_1005Metric; LCSC Part C19666 -> C726612
- R1: renamed from R3; LCSC Part C105637 -> C25867
- R2: renamed from R11; LCSC Part C105637 -> C25900
- R3: renamed from R15; LCSC Part C105637 -> C25900
- R4: renamed from R2; LCSC Part C105637 -> C407753
- R5: renamed from R12; LCSC Part C105637 -> C25792
- R6: renamed from R13; LCSC Part C105637 -> C25871
- R7: renamed from R14; LCSC Part C105637 -> C407753
- R8: renamed from R7; LCSC Part C105872 -> C25905
- R9: renamed from R10; LCSC Part C105872 -> C25905
- Y1: value 32.768 kHz -> 32MHz; footprint easyeda2kicad:FC-135R_L3.2-W1.5 -> Crystal:Crystal_SMD_2016-4Pin_2.0x1.6mm; LCSC Part C32346 -> C255896
- renumbered E2 to E1, J3 to J1, J1 to J2, J4 to J3, J5 to J4, J2 to J5, Q2 to Q1, SW89 to SW90, U6 to U2, U5 to U3, U7 to U4
Connections:
- net TSENS is gone; now on an unnamed net: U2.1 (TS)
- net ConnD+: now also U1.AD6 (D+)
- net ConnD-: now also U1.AD4 (D-)
- net ConnVBUS: now also C19.1, C21.1, U1.AD2 (VBUS); no longer C6.1
- net GND: now also C1.1, C10.1, C5.1, C9.1, U2.15 (SYSOFF), C11.1, C12.2, C13.1, C14.1, C15.2, C16.2, C17.1, C18.1, C19.2, C20.2, C21.2, C22.2, C23.2, C24.2, C25.2, C26.1, U1.74 (GND), U1.B7 (VSS), U1.F23 (VSS_PA); no longer C1.2, C10.2, C5.2, C9.2
- net SWCLK: now also U1.AA24 (SWDCLK)
- net SWDIO: now also U1.AC24 (SWDIO)
- net SYS_PWR: now also D1.2 (A), U2.10 (OUT), U2.11 (OUT), C23.1, C24.1; no longer C9.1
- net VBAT: now also C26.2; no longer C1.1, C8.1
- net VDD_NRF: now also C6.1, C7.1, C8.1, C12.1, C14.2, C25.1, U1.A22 (VDD), U1.AD14 (VDD), U1.AD23 (VDD), U1.B1 (VDD), U1.W1 (VDD), U1.Y2 (VDDH); no longer C10.1, C4.1
- net at Y1.1: now also C2.2, U1.A23 (XC2); no longer C5.1
- net at C3.1: now also L1.1, U1.H23 (ANT)
- net at Y1.2: now also C1.2, U1.B24 (XC1); no longer C2.2
- removed net SYS_POWER: C7.1, D1.2 (A), U2.10 (OUT), U2.11 (OUT)
- new net: C10.2, C15.1, C16.1, L3.1, U1.B5 (DEC4), U1.E24 (DEC6)
- new net: C13.2, U1.A18 (DEC2)
- new net: C17.2, U1.D2 (P0.00/XL1), Y2.1
- new net: C18.2, U1.F2 (P0.01/XL2), Y2.2
- new net: C22.1, C4.1, L1.2
- new net: L2.1, L3.2
- new net: C20.1, U1.AC5 (DECUSB)
- new net: L2.2, U1.B3 (DCC)
- new net: C5.2, U1.C1 (DEC1)
- new net: C11.2, U1.D23 (DEC3)
- new net: C9.2, U1.N24 (DEC5)
- no-connect marks 18 -> 13
Other:
- note added: "MCU nRF52840"
- note added: "not req for Fxx and later"
- note removed: "MCU nRF52840 MDBT50Q-U1MV2"
- note removed: "NTC Selector"
- note removed: "Power & Battery Status"
- note removed: "Voltage Regulator"
- note removed: "check if footprint pins are correct!!!!"
- moved on the sheet: BT1, D1, E1, J1, J2, J3, J4, J5, Q1, R1, R2, R3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

Commit message: update lolololololololo
Parts:
- added U5: BQ25188YBGR_C43043524, easyeda2kicad:WCSP-8_L1.6-W1.0-P0.40-TL_IS31FL3194-CLS2, symbol easyeda2kicad:BQ25188YBGR_C43043524
- added U6: MAX17048G+T10, easyeda2kicad:TDFN-8_L2.0-W2.0-P0.50-BL-EP1.2, symbol easyeda2kicad:MAX17048G+T10
- added U7: TPS62840DLCR, easyeda2kicad:VSON-8_L2.0-W1.5-P0.50-BL, symbol easyeda2kicad:TPS62840DLCR
- U1: value ~ -> NRF52840
Connections:
- net SCL: now also U5.B1 (SCL), U6.7 (SCL)
- net SDA: now also U5.C1 (SDA), U6.8 (SDA)
Other:
- moved on the sheet: C19, C23, C24, C25, C26, D1, R1, R2, R3, R4, R5, R6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

Commit message: update
Parts:
- removed U6: MAX17048G+T10, easyeda2kicad:TDFN-8_L2.0-W2.0-P0.50-BL-EP1.2, symbol easyeda2kicad:MAX17048G+T10
Connections:
- net ConnVBUS: now also U5.A2 (IN)
- net SYS_PWR: now also U5.B2 (SYS)
- net /INT: now reaches U5.A1 (/INT)
Other:
- moved on the sheet: U7

Commit message: update - change pmic to npm1300
Parts:
- added C27, C32, C33: 1u, Capacitor_SMD:C_0603_1608Metric, symbol Device:C_Small
- added C28: 2.2u, Capacitor_SMD:C_0603_1608Metric, symbol Device:C_Small
- added C29, C30, C31: 10u, Capacitor_SMD:C_0603_1608Metric, symbol Device:C_Small
- added D2: LED_RGB, symbol Device:LED_RGB
- added L4: 2.2u, Inductor_SMD:L_0402_1005Metric, symbol Device:L_Small
- added R10: 470k, Resistor_SMD:R_0402_1005Metric, symbol Device:R_Small
- added U?: ${ALTIUM_VALUE}, Nordic_QFN50P500X500X90-33N:Nordic_QFN50P500X500X90-33N, symbol AltiumLib:root_0_nPM1300_QEAA_AltiumLib.DbLib
Connections:
- net ConnVBUS: now also C27.1, U?.21 (VBUS)
- net GND: now also C27.2, C28.2, C29.2, C30.2, C31.2, C32.2, C33.2, R10.2, U?.17 (VSET1), U?.2 (PVSS1), U?.30 (LSIN2/VINLDO2), U?.31 (LSOUT2/VOUTLDO2), U?.33 (AVSS), U?.6 (PVSS2)
- net SCL: now also U?.14 (SCL)
- net SDA: now also U?.13 (SDA)
- net VBAT: now also C28.1, U?.19 (VBAT)
- net VDD_NRF: now also C29.1, L4.1, U?.28 (LSIN1/VINLDO1), U?.32 (VOUT2)
- new net: D2.1 (RK), U?.25 (LED0)
- new net: D2.2 (GK), U?.26 (LED1)
- new net: D2.3 (BK), U?.27 (LED2)
- new net: R10.1, U?.16 (VSET2)
- new net: C33.1, U?.29 (LSOUT1/VOUTLDO1)
- new net: L4.2, U?.5 (SW2)
- new net VBUSOUT: C32.1, U?.22 (VBUSOUT)
- new net VSYS: C30.1, C31.1, D2.4 (BA), D2.5 (GA), D2.6 (RA), U?.1 (VOUT1), U?.20 (VSYS), U?.4 (PVDD)
- no-connect marks 13 -> 21
Other:
- note added: "Li-ion, Li-polymer, or LiFePO4"
- note added: "TBD!!!"
- note added: "ogarnac jak je podpiac"
- moved on the sheet: BT1, E1, J1, J2, J3, J4, J5, Q1, R8, R9, SW90, U5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

Commit message: update
Parts:
- removed C19, C23, C24, C25: 4.7u, Capacitor_SMD:C_0603_1608Metric, symbol Device:C_Small
- removed C26: 1u, Capacitor_SMD:C_0603_1608Metric, symbol Device:C_Small
- removed D1: Red, LED_SMD:LED_0201_0603Metric, symbol Device:LED_Small
- removed R2, R3: 4.7k, Resistor_SMD:R_0402_1005Metric, symbol Device:R_Small
- removed R4, R7: 10k, Resistor_SMD:R_0402_1005Metric, symbol Device:R_Small
- removed R5: 47k, Resistor_SMD:R_0402_1005Metric, symbol Device:R_Small
- removed R6: 1.8k, Resistor_SMD:R_0402_1005Metric, symbol Device:R_Small
- removed U2: BQ24075RGTR, easyeda2kicad:QFN-16_L3.0-W3.0-P0.50-TL-EP1.7, symbol easyeda2kicad:BQ24075RGTR
- removed U3: XC6220B331ER-G, easyeda2kicad:USP-6C_L2.0-W1.8-P0.50-BL-EP, symbol easyeda2kicad:XC6220B331ER-G
- removed U4: LC709203FXE-03MH, easyeda2kicad:WLCSP-9_L1.6-W1.8-R3-C3-P0.50-BL, symbol easyeda2kicad:LC709203FXE-03MH
- removed U5: BQ25188YBGR_C43043524, easyeda2kicad:WCSP-8_L1.6-W1.0-P0.40-TL_IS31FL3194-CLS2, symbol easyeda2kicad:BQ25188YBGR_C43043524
- removed U7: TPS62840DLCR, easyeda2kicad:VSON-8_L2.0-W1.5-P0.50-BL, symbol easyeda2kicad:TPS62840DLCR
- added JP1: SolderJumper_2_Open, symbol Jumper:SolderJumper_2_Open
- added NTC1: Conn_01x01_Socket, symbol Connector:Conn_01x01_Socket
- BT1: LCSC Part (none) -> -
- C28: LCSC Part C559769 -> C309478
- C29, C30, C31: LCSC Part C277476 -> C596327
- D2: footprint (none) -> easyeda2kicad:LED-SMD_4P-L1.6-W1.5-TR-1; symbol Device:LED_RGB -> Device:LED_RGBA; LCSC Part (none) -> C3029071
- L4: footprint Inductor_SMD:L_0402_1005Metric -> Inductor_SMD:L_1008_2520Metric; LCSC Part C304335 -> C5349606
- R1: value 1.5k -> 10k; LCSC Part C25867 -> C25744
- U2: renamed from U?; value ${ALTIUM_VALUE} -> nPM1300-QEAA; LCSC Part (none) -> C7466043
Connections:
- net ConnVBUS: no longer C21.1, U1.AD2 (VBUS)
- net GND: now also R1.1
- net VBUSOUT: now also C21.1, U1.AD2 (VBUS)
- net VDD_NRF: now also U2.12 (VDDIO)
- net VSYS: no longer D2.5 (GA), D2.6 (RA)
- net at R1.2: now also JP1.1 (A)
- net CC1: now reaches R8.2, USBC1.A5 (CC1)
- net CC1: now also U2.23 (CC1)
- net CC2: now reaches R9.2, USBC1.B5 (CC2)
- net CC2: now also U2.24 (CC2)
- net at U2.18 (NTC): now also JP1.2 (B), NTC1.1 (Pin_1)
- no-connect marks 21 -> 15
Other:
- note removed: "3V3 LDO Regulator"
- note removed: "Battery Fuel Gauge"
- note removed: "Power Path & Charger"
- note removed: "ogarnac jak je podpiac"

Commit message: update - pcb layout
Changed lines of the file:
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@@
 	(text "not req for Fxx and later"
 		(exclude_from_sim no)
-		(at 145.288 88.9 0)
+		(at 150.368 89.408 0)
 		(effects
 			(font

Commit message: update
Parts:
- removed Q1: DMP2123LQ, easyeda2kicad:SOT-23-3_L2.9-W1.3-P1.90-LS2.4-BR, symbol easyeda2kicad:DMP2123LQ
- added J6: Conn_Coaxial_Small, easyeda2kicad:IPEX-SMD_3P-L2.6-W2.6-LS3.0_ZCF-CF0001-0002IPEX, symbol Connector:Conn_Coaxial_Small
- added Q1: PMZB350UPE,315, Package_DFN_QFN:Diodes_DFN1006-3, symbol Device:Q_PMOS
- JP1: footprint (none) -> Jumper:SolderJumper-2_P1.3mm_Open_RoundedPad1.0x1.5mm
- Yr1: renamed from Y1; symbol Device:Crystal_Small -> Device:Crystal_GND24_Small
Connections:
- net GND: now also Yr1.2 (G), Yr1.4 (G), J6.2 (Ext), Q1.G
- net VBAT: now also Q1.D
- net at C17.2, U1.D2 (P0.00/XL1): now also Y2.2; no longer Y2.1
- net at C18.2, U1.F2 (P0.01/XL2): now also Y2.1; no longer Y2.2
- net at C22.1, C4.1, L1.2: now also J6.1 (In)
- net at C1.2, U1.B24 (XC1): now also Yr1.3; no longer Yr1.2
- net at J2.1: now also Q1.S
Changed lines of the file:
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@@
 	(wire
 		(pts
-			(xy 176.53 215.9) (xy 172.72 215.9)
+			(xy 148.59 78.74) (xy 148.59 81.28)
 		)
 		(stroke
@@
 	(wire
 		(pts
-			(xy 148.59 78.74) (xy 148.59 81.28)
+			(xy 110.49 48.26) (xy 110.49 50.8)
 		)
 		(stroke
@@
 	(wire
 		(pts
-			(xy 110.49 48.26) (xy 110.49 50.8)
+			(xy 93.98 35.56) (xy 93.98 36.83)
 		)
 		(stroke
@@
 	(wire
 		(pts
-			(xy 93.98 35.56) (xy 93.98 36.83)
+			(xy 184.15 76.2) (xy 185.42 76.2)
 		)
 		(stroke
@@
 	(wire
 		(pts
+			(xy 172.72 215.9) (xy 173.99 215.9)
+		)
+		(stroke
+			(width 0)
+			(type default)
+		)
+	)
+	(wire
+		(pts
 			(xy 156.21 41.91) (xy 156.21 39.37)
 		)
@@
 	(wire
 		(pts
+			(xy 152.4 39.37) (xy 152.4 46.99)
+		)
+		(stroke
+			(width 0)
+			(type default)
+		)
+	)
+	(wire
+		(pts
 			(xy 54.61 104.14) (xy 57.15 104.14)
 		)
@@
 	(wire
 		(pts
+			(xy 185.42 76.2) (xy 185.42 81.28)
+		)
+		(stroke
+			(width 0)
+			(type default)
+		)
+	)
+	(wire
+		(pts
 			(xy 17.78 68.58) (xy 20.32 68.58)
 		)
@@
 			)
 		)
-		(property "Footprint" ""
+		(property "Footprint" "Jumper:SolderJumper-2_P1.3mm_Open_RoundedPad1.0x1.5mm"
 			(at 226.06 69.85 0)
 			(effects
@@
 		(lib_id "Device:Crystal_Small")
 		(at 27.94 72.39 270)
+		(mirror x)
 		(unit 1)
 		(exclude_from_sim no)
@@
 		(dnp no)
 		(property "Reference" "Y2"
-			(at 30.48 71.1199 90)
+			(at 30.48 73.6601 90)
 			(effects
 				(font
@@
 		)
 		(property "Value" "32.768 kHz"
-			(at 30.48 73.6599 90)
+			(at 30.48 71.1201 90)
 			(effects
 				(font
@@
 	)
 	(symbol
+		(lib_id "Device:Q_PMOS")
+		(at 179.07 215.9 0)
+		(unit 1)
+		(exclude_from_sim no)
+		(in_bom yes)
+		(on_board yes)
+		(dnp no)
+		(property "Reference" "Q1"
+			(at 185.42 214.6299 0)
+			(effects
+				(font
+					(size 1.27 1.27)
+				)
+				(justify left)
+			)
+		)
+		(property "Value" "PMZB350UPE,315"
+			(at 185.42 217.1699 0)
+			(effects
+				(font
+					(size 0.889 0.889)
+				)
+				(justify left)
+			)
+		)
+		(property "Footprint" "Package_DFN_QFN:Diodes_DFN1006-3"
+			(at 184.15 213.36 0)
+			(effects
+				(font
+					(size 1.27 1.27)
+				)
+				(hide yes)
+			)
+		)
+		(property "Datasheet" "https://www.lcsc.com/product-detail/C478140.html"
+			(at 179.07 215.9 0)
+			(effects
+				(font
+					(size 1.27 1.27)
+				)
+				(hide yes)
+			)
+		)
+		(property "Description" "P-MOSFET transistor"
+			(at 179.07 215.9 0)
+			(effects
+				(font
+					(size 1.27 1.27)
+				)
+				(hide yes)
+			)
+		)
+		(property "LCSC Part" "C478140"
+			(at 179.07 215.9 0)
+			(effects
+				(font
+					(size 1.27 1.27)
+				)
+				(hide yes)
+			)
+		)
+		(pin "D"
+		)
+		(pin "G"
+		)
+		(pin "S"
+		)
+		(instances
+			(project ""
+				(path "/17f6a4a5-fbff-4e30-a1cc-9481373e4968"
+					(reference "Q1")
+					(unit 1)
+				)
+			)
+		)
+	)
+	(symbol
 		(lib_id "easyeda2kicad:726386-2")
 		(at 80.01 267.97 180)
@@
 	)
 	(symbol
+		(lib_id "Connector:Conn_Coaxial_Small")
+		(at 181.61 76.2 0)
+		(unit 1)
+		(exclude_from_sim no)
+		(in_bom yes)
+		(on_board yes)
+		(dnp no)
+		(property "Reference" "J6"
+			(at 181.61 73.152 0)
+			(effects
+				(font
+					(size 1.27 1.27)
+				)
+			)
+		)
+		(property "Value" "Conn_Coaxial_Small"
+			(at 181.0904 72.39 0)
+			(effects
+				(font
+					(size 1.27 1.27)
+				)
+				(hide yes)
+			)
+		)
+		(property "Footprint" "easyeda2kicad:IPEX-SMD_3P-L2.6-W2.6-LS3.0_ZCF-CF0001-0002IPEX"
+			(at 181.61 76.2 0)
+			(effects
+				(font
+					(size 1.27 1.27)
+				)
+				(hide yes)
+			)
+		)
+		(property "Datasheet" "~"
+			(at 181.61 76.2 0)
+			(effects
+				(font
+					(size 1.27 1.27)
+				)
+				(hide yes)
+			)
+		)
+		(property "Description" "small coaxial connector (BNC, SMA, SMB, SMC, Cinch/RCA, LEMO, ...)"
+			(at 181.61 76.2 0)
+			(effects
+				(font
+					(size 1.27 1.27)
+				)
+				(hide yes)
+			)
+		)
+		(pin "1"
+		)
+		(pin "2"
+		)
+		(instances
+			(project ""
+				(path "/17f6a4a5-fbff-4e30-a1cc-9481373e4968"
+					(reference "J6")
+					(unit 1)
+				)
+			)
+		)
+	)
+	(symbol
 		(lib_id "Device:C_Small")
 		(at 140.97 71.12 270)
@@
 	(symbol
 		(lib_id "power:GND")
-		(at 318.77 105.41 0)
+		(at 185.42 81.28 0)
 		(mirror y)
 		(unit 1)
@@
 		(dnp no)
 		(fields_autoplaced yes)
-		(property "Reference" "#PWR025"
-			(at 318.77 111.76 0)
+		(property "Reference" "#PWR020"
+			(at 185.42 87.63 0)
 			(effects
 				(font
@@
 		)
 		(property "Value" "GND"
-			(at 318.77 110.49 0)
+			(at 185.42 86.36 0)
 			(effects
 				(font
@@
 		)
 		(property "Footprint" ""
-			(at 318.77 105.41 0)
+			(at 185.42 81.28 0)
 			(effects
 				(font
@@
 		)
 		(property "Datasheet" ""
-			(at 318.77 105.41 0)
+			(at 185.42 81.28 0)
 			(effects
 				(font
@@
 		)
 		(property "Description" "Power symbol creates a global label with name \"GND\" , ground"
-			(at 318.77 105.41 0)
+			(at 185.42 81.28 0)
 			(effects
 				(font
@@
 			(project "ibm-modern-m-ssk"
 				(path "/17f6a4a5-fbff-4e30-a1cc-9481373e4968"
-					(reference "#PWR025")
+					(reference "#PWR020")
 					(unit 1)
 				)
@@
 	)
 	(symbol
-		(lib_id "easyeda2kicad:DMP2123LQ")
-		(at 181.61 215.9 0)
+		(lib_id "power:GND")
+		(at 318.77 105.41 0)
+		(mirror y)
 		(unit 1)
 		(exclude_from_sim no)
@@
 		(on_board yes)
 		(dnp no)
-		(property "Reference" "Q1"
-			(at 185.166 212.344 0)
-			(effects
-				(font
-					(size 1.27 1.27)
-				)
-				(justify left)
-			)
-		)
-		(property "Value" "DMP2123LQ"
-			(at 185.166 214.122 0)
-			(effects
-				(font
-					(size 1.27 1.27)
-				)
-				(justify left)
-			)
-		)
-		(property "Footprint" "easyeda2kicad:SOT-23-3_L2.9-W1.3-P1.90-LS2.4-BR"
-			(at 181.61 228.6 0)
+		(fields_autoplaced yes)
+		(property "Reference" "#PWR025"
+			(at 318.77 111.76 0)
 			(effects
 				(font
@@
 			)
 		)
-		(property "Datasheet" "https://www.lcsc.com/product-detail/C3647032.html"
-			(at 181.61 215.9 0)
+		(property "Value" "GND"
+			(at 318.77 110.49 0)
 			(effects
 				(font
@@
 			)
 		)
-		(property "Description" ""
-			(at 181.61 215.9 0)
+		(property "Footprint" ""
+			(at 318.77 105.41 0)
 			(effects
 				(font
@@
 			)
 		)
-		(property "LCSC Part" "C3647032"
-			(at 181.61 231.14 0)
+		(property "Datasheet" ""
+			(at 318.77 105.41 0)
 			(effects
 				(font
@@
 			)
 		)
-		(property "Sim.Pin" ""
-			(at 181.61 215.9 0)
+		(property "Description" "Power symbol creates a global label with name \"GND\" , ground"
+			(at 318.77 105.41 0)
 			(effects
 				(font
@@
 			)
 		)
-		(pin "2"
-		)
 		(pin "1"
 		)
-		(pin "3"
-		)
 		(instances
 			(project "ibm-modern-m-ssk"
 				(path "/17f6a4a5-fbff-4e30-a1cc-9481373e4968"
-					(reference "Q1")
+					(reference "#PWR025")
 					(unit 1)
 				)
@@
 	)
 	(symbol
-		(lib_id "Device:Crystal_Small")
+		(lib_id "Device:Crystal_GND24_Small")
 		(at 152.4 49.53 0)
 		(mirror x)
@@
 		(on_board yes)
 		(dnp no)
-		(property "Reference" "Y1"
+		(property "Reference" "Yr1"
 			(at 151.1299 52.07 90)
 			(effects
@@
 			)
 		)
-		(property "Datasheet" ""
+		(property "Datasheet" "~"
 			(at 152.4 49.53 0)
 			(effects
@@
 			)
 		)
-		(property "Description" "Two pin crystal, small symbol"
+		(property "Description" "Four pin crystal, GND on pins 2 and 4, small symbol"
 			(at 152.4 49.53 0)
 			(effects
@@
 		(pin "2"
 		)
+		(pin "4"
+		)
+		(pin "3"
+		)
 		(instances
 			(project "ibm-modern-m-ssk"
 				(path "/17f6a4a5-fbff-4e30-a1cc-9481373e4968"
-					(reference "Y1")
+					(reference "Yr1")
 					(unit 1)
 				)
