File: kicad/ibm-modern-m-ssk.kicad_sch (KiCad schematic)
At the start: 54 parts, among them J1 TF38-24S-0.5SV(830), J2 S2B-PH-SM4-TB(LF)(SN), J3 Conn_02x06_Odd_Even, J4 Conn_01x04_Pin, J5 726386-2, J6 Conn_Coaxial_Small, Q1 PMZB350UPE,315, SW90 SW_Push, U1 NRF52840, U2 nPM1300-QEAA, Y2 32.768 kHz

Commit message: update
Parts:
- removed JP1: SolderJumper_2_Open, Jumper:SolderJumper-2_P1.3mm_Open_RoundedPad1.0x1.5mm, symbol Jumper:SolderJumper_2_Open
- removed NTC1: Conn_01x01_Socket, symbol Connector:Conn_01x01_Socket
- BT1: value Li-Po 603450 -> LP803040; footprint easyeda2kicad:LiPo_603450 -> easyeda2kicad:LP803040
- J2: value S2B-PH-SM4-TB(LF)(SN) -> Molex PicoBlade; footprint easyeda2kicad:CONN-SMD_2P-P1.00_SM02B-SRSS-TB-LF-SN -> Connector_Molex:Molex_PicoBlade_53261-0271_1x02-1MP_P1.25mm_Horizontal; LCSC Part C160402 -> C177225
Connections:
- net GND: now also Q1.1 (G); no longer Q1.G
- net VBAT: now also Q1.3 (D); no longer Q1.D
- net at U2.18 (NTC): now also R1.2
- net at J2.1: now also Q1.2 (S); no longer Q1.S
Other:
- note removed: "(only for 3d model)"
Changed lines of the file:
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@@
 		)
 	)
-	(text "(only for 3d model)"
-		(exclude_from_sim no)
-		(at 178.816 279.908 0)
-		(effects
-			(font
-				(size 0.762 0.762)
-				(thickness 0.3048)
-				(bold yes)
-			)
-			(justify left)
-		)
-	)
 	(text "Battery"
 		(exclude_from_sim no)
-		(at 178.562 277.876 0)
+		(at 178.308 279.4 0)
 		(effects
 			(font
@@
 	)
 	(junction
-		(at 226.06 66.04)
-		(diameter 0)
-		(color 0 0 0 0)
-	)
-	(junction
 		(at 306.07 93.98)
 		(diameter 0)
@@
 	(wire
 		(pts
+			(xy 226.06 66.04) (xy 226.06 73.66)
+		)
+		(stroke
+			(width 0)
+			(type default)
+		)
+	)
+	(wire
+		(pts
 			(xy 66.04 134.62) (xy 67.31 134.62)
 		)
@@
 	)
 	(symbol
-		(lib_id "Connector:Conn_01x01_Socket")
-		(at 220.98 66.04 180)
-		(unit 1)
-		(exclude_from_sim no)
-		(in_bom yes)
-		(on_board yes)
-		(dnp no)
-		(property "Reference" "NTC1"
-			(at 219.456 66.04 0)
-			(effects
-				(font
-					(size 0.889 0.889)
-				)
-			)
-		)
-		(property "Value" "Conn_01x01_Socket"
-			(at 221.615 63.5 0)
-			(effects
-				(font
-					(size 1.27 1.27)
-				)
-				(hide yes)
-			)
-		)
-		(property "Footprint" ""
-			(at 220.98 66.04 0)
-			(effects
-				(font
-					(size 1.27 1.27)
-				)
-				(hide yes)
-			)
-		)
-		(property "Datasheet" "~"
-			(at 220.98 66.04 0)
-			(effects
-				(font
-					(size 1.27 1.27)
-				)
-				(hide yes)
-			)
-		)
-		(property "Description" "Generic connector, single row, 01x01, script generated"
-			(at 220.98 66.04 0)
-			(effects
-				(font
-					(size 1.27 1.27)
-				)
-				(hide yes)
-			)
-		)
-		(pin "1"
-		)
-		(instances
-			(project ""
-				(path "/17f6a4a5-fbff-4e30-a1cc-9481373e4968"
-					(reference "NTC1")
-					(unit 1)
-				)
-			)
-		)
-	)
-	(symbol
 		(lib_id "Device:C_Small")
 		(at 121.92 45.72 0)
@@
 	)
 	(symbol
-		(lib_id "Jumper:SolderJumper_2_Open")
-		(at 226.06 69.85 90)
-		(unit 1)
-		(exclude_from_sim no)
-		(in_bom no)
-		(on_board yes)
-		(dnp no)
-		(property "Reference" "JP1"
-			(at 227.584 70.104 90)
-			(effects
-				(font
-					(size 0.889 0.889)
-				)
-				(justify right)
-			)
-		)
-		(property "Value" "SolderJumper_2_Open"
-			(at 228.6 71.1199 90)
-			(effects
-				(font
-					(size 1.27 1.27)
-				)
-				(justify right)
-				(hide yes)
-			)
-		)
-		(property "Footprint" "Jumper:SolderJumper-2_P1.3mm_Open_RoundedPad1.0x1.5mm"
-			(at 226.06 69.85 0)
-			(effects
-				(font
-					(size 1.27 1.27)
-				)
-				(hide yes)
-			)
-		)
-		(property "Datasheet" "~"
-			(at 226.06 69.85 0)
-			(effects
-				(font
-					(size 1.27 1.27)
-				)
-				(hide yes)
-			)
-		)
-		(property "Description" "Solder Jumper, 2-pole, open"
-			(at 226.06 69.85 0)
-			(effects
-				(font
-					(size 1.27 1.27)
-				)
-				(hide yes)
-			)
-		)
-		(pin "1"
-		)
-		(pin "2"
-		)
-		(instances
-			(project ""
-				(path "/17f6a4a5-fbff-4e30-a1cc-9481373e4968"
-					(reference "JP1")
-					(unit 1)
-				)
-			)
-		)
-	)
-	(symbol
 		(lib_id "power:GND")
 		(at 312.42 55.88 0)
@@
 			)
 		)
-		(pin "D"
+		(pin "2"
 		)
-		(pin "G"
+		(pin "1"
 		)
-		(pin "S"
+		(pin "3"
 		)
 		(instances
@@
 			)
 		)
-		(property "Value" "S2B-PH-SM4-TB(LF)(SN)"
+		(property "Value" "Molex PicoBlade"
 			(at 180.34 240.03 90)
 			(effects
@@
 			)
 		)
-		(property "Footprint" "easyeda2kicad:CONN-SMD_2P-P1.00_SM02B-SRSS-TB-LF-SN"
+		(property "Footprint" "Connector_Molex:Molex_PicoBlade_53261-0271_1x02-1MP_P1.25mm_Horizontal"
 			(at 166.37 228.6 0)
 			(effects
@@
 			)
 		)
-		(property "Datasheet" "https://www.lcsc.com/product-detail/C160402.html"
+		(property "Datasheet" "https://www.lcsc.com/product-detail/C177225.html"
 			(at 163.83 228.6 0)
 			(effects
@@
 			)
 		)
-		(property "LCSC Part" "C160402"
+		(property "LCSC Part" "C177225"
 			(at 161.29 228.6 0)
 			(effects
@@
 			)
 		)
-		(property "Value" "Li-Po 603450"
+		(property "Value" "LP803040"
 			(at 189.9285 262.89 90)
 			(effects
@@
 			)
 		)
-		(property "Footprint" "easyeda2kicad:LiPo_603450"
+		(property "Footprint" "easyeda2kicad:LP803040"
 			(at 190.246 267.97 90)
 			(effects
@@
 			)
 		)
-		(property "Datasheet" "~"
+		(property "Datasheet" "https://www.tme.eu/Document/8518e6f80c7c95dc96792c6f2286ce95/aky2417.pdf"
 			(at 190.246 267.97 90)
 			(effects
