File: kicad/ibm-modern-m-ssk.kicad_sch (KiCad schematic)
At the start: 52 parts, among them J1 TF38-24S-0.5SV(830), J2 Molex PicoBlade, J3 Conn_02x06_Odd_Even, J4 Conn_01x04_Pin, J5 726386-2, J6 Conn_Coaxial_Small, Q1 PMZB350UPE,315, SW90 SW_Push, U1 NRF52840, U2 nPM1300-QEAA, Y2 32.768 kHz

Commit message: update
Parts:
- removed E1: TPD2E001DRYR-TP, easyeda2kicad:SON-6_L1.4-W1.0-P0.50-TL_USBULC6-2M6, symbol easyeda2kicad:TPD2E001DRYR-TP
- added D1: PESDNC2FD5VB, easyeda2kicad:Diodes_DFN1006-2, symbol Device:D_TVS_Small
- added F1: BSMD0603L-150, Fuse:Fuse_0603_1608Metric, symbol Device:Polyfuse
- added J8: Conn_01x08_MountingPin, Connector_FFC-FPC:Amphenol_F32Q-1A7x1-11008_1x08-1MP_P0.5mm_Horizontal, symbol Connector_Generic_MountingPin:Conn_01x08_MountingPin
- added U3: TPD4E05U06DQAR, Package_SON:USON-10_2.5x1.0mm_P0.5mm, symbol Power_Protection:TPD4E05U06DQA
- renumbered USBC1 to J1, J1 to J7
Connections:
- net CC1: now also U3.1 (D1+), U3.10 (NC); no longer R8.2
- net CC2: now also U3.5 (D2-), U3.6 (NC); no longer R9.2
- net GND: now also D1.1 (A1), U3.3 (GND), U3.8 (GND); no longer R8.1, R9.1
- net ConnD+ renamed D+
- net D+: now also U3.4 (D2+), U3.7 (NC)
- net ConnD- renamed D-
- net D-: now also U3.2 (D1-), U3.9 (NC)
- net ConnVBUS renamed VBUS
- net VBUS: now also F1.1
- new net VCOM: D1.2 (A2), F1.2
- no-connect marks 15 -> 13
Other:
- moved on the sheet: J1, J2, J7, Q1, R8, R9

Commit message: update
Parts:
- removed D2: LED_RGB, easyeda2kicad:LED-SMD_4P-L1.6-W1.5-TR-1, symbol Device:LED_RGBA
- removed J1: TYPE-C-31-M-12, easyeda2kicad:USB-C_SMD-TYPE-C-31-M-12_1, symbol easyeda2kicad:TYPE-C-31-M-12
- removed J8: Conn_01x08_MountingPin, Connector_FFC-FPC:Amphenol_F32Q-1A7x1-11008_1x08-1MP_P0.5mm_Horizontal, symbol Connector_Generic_MountingPin:Conn_01x08_MountingPin
- removed R1: 10k, Resistor_SMD:R_0402_1005Metric, symbol Device:R_Small
- removed R8, R9: 5.1k, Resistor_SMD:R_0402_1005Metric, symbol Device:R_Small
- added D4, D92: rgb, LED_SMD:LED_Wurth_150044M155260, symbol easyeda2kicad:rgb
- added J1: TYPE-C-31-D-06, easyeda2kicad:USB-C-SMD_TYPE-C-31-D-06, symbol Connector:USB_C_Receptacle_USB2.0_16P
- added J8: FPC_12P_0.5mm, easyeda2kicad:FPC_12P_0.5mm, symbol Connector_Generic:Conn_01x12
- added J9: FH12-12S-0.5SVA(54), easyeda2kicad:FH1212S05SVA54, symbol Connector_Generic_MountingPin:Conn_01x12_MountingPin
- added SW89, SW91: SW_Push, easyeda2kicad:SW-SMD_2P-L3.0-W2.5-LS4.0, symbol Switch:SW_Push
- added TH1: 10k, symbol Device:Thermistor_NTC
Connections:
- net VCOM is gone; now on net VBUS: D1.2 (A2), F1.2
- net CC1: now also J1.A5 (CC1), J8.4 (Pin_4), J9.4 (Pin_4)
- net CC2: now also J1.B5 (CC2), J8.9 (Pin_9), J9.9 (Pin_9)
- net D+: now also U3.2 (D1-), U3.9 (NC), J1.A6 (D+), J1.B6 (D+), J8.6 (Pin_6), J9.6 (Pin_6); no longer U3.4 (D2+), U3.7 (NC)
- net D-: now also U3.4 (D2+), U3.7 (NC), J1.A7 (D-), J1.B7 (D-), J8.7 (Pin_7), J9.7 (Pin_7); no longer U3.2 (D1-), U3.9 (NC)
- net GND: now also Q1.G, U2.16 (VSET2), D4.2 (VSS), D92.2 (VSS), J1.A1 (GND), J1.A12 (GND), J1.B1 (GND), J1.B12 (GND), J1.S1 (SHIELD), J8.5 (Pin_5), J8.8 (Pin_8), J9.5 (Pin_5), J9.8 (Pin_8), SW89.2, SW91.2, TH1.2; no longer C29.2, C30.2, Q1.1 (G), U2.17 (VSET1), U2.2 (PVSS1), Yr1.4 (G)
- net VBAT: now also Q1.D; no longer Q1.3 (D)
- net VBUS: now also J8.1 (Pin_1), J8.2 (Pin_2), J9.1 (Pin_1), J9.2 (Pin_2); no longer F1.1
- net VDD_NRF: now also U2.1 (VOUT1); no longer U2.12 (VDDIO), U2.32 (VOUT2)
- net VSYS: now also U2.32 (VOUT2), D4.4 (VDD), D92.4 (VDD), J8.12 (Pin_12), J9.12 (Pin_12); no longer U2.1 (VOUT1)
- net at U2.18 (NTC): now also TH1.1
- net at R10.1: now also U2.17 (VSET1); no longer U2.16 (VSET2)
- net at J2.1: now also Q1.S; no longer Q1.2 (S)
- net at L4.2: now also U2.3 (SW1); no longer U2.5 (SW2)
- net SHPHLD: now reaches U2.15 (SHPHLD)
- net SHPHLD: now also J8.11 (Pin_11), J9.11 (Pin_11), SW91.1
- new net: F1.1, J1.A4 (VBUS), J1.A9 (VBUS), J1.B4 (VBUS), J1.B9 (VBUS)
- new net: D4.1 (DOUT), D92.3 (DIN)
- new net BT_PAIR: J8.3 (Pin_3), J9.3 (Pin_3), SW89.1
- new net LED_DATA: D4.3 (DIN), J8.10 (Pin_10), J9.10 (Pin_10)
- new net PVSS1: C29.2, C30.2, U2.2 (PVSS1)
- no-connect marks 13 -> 18
Other:
- note added: "Via to GND-layer on PVSS1"
- note removed: "ESD Protection"
- note removed: "USB C"
- moved on the sheet: C29, C33, D1, F1, L4, R10

Commit message: update
Parts:
- removed BT1: LP803040, easyeda2kicad:LP803040, symbol Device:Battery_Cell
- removed C1, C17, C18, C2: 12p, Capacitor_SMD:C_0402_1005Metric, symbol Device:C_Small
- removed C10, C13, C22: NC, Capacitor_SMD:C_0402_1005Metric, symbol Device:C_Small
- removed C11: 100p, Capacitor_SMD:C_0402_1005Metric, symbol Device:C_Small
- removed C12, C5, C7, C8: 100n, Capacitor_SMD:C_0402_1005Metric, symbol Device:C_Small
- removed C14, C15, C27, C32, C33: 1u, Capacitor_SMD:C_0603_1608Metric, symbol Device:C_Small
- removed C16: 47n, Capacitor_SMD:C_0402_1005Metric, symbol Device:C_Small
- removed C20, C21, C6: 4.7u, Capacitor_SMD:C_0603_1608Metric, symbol Device:C_Small
- removed C28: 2.2u, Capacitor_SMD:C_0603_1608Metric, symbol Device:C_Small
- removed C29, C30, C31: 10u, Capacitor_SMD:C_0603_1608Metric, symbol Device:C_Small
- removed C3: 0.8p, Capacitor_SMD:C_0402_1005Metric, symbol Device:C_Small
- removed C4: 0.5p, Capacitor_SMD:C_0402_1005Metric, symbol Device:C_Small
- removed C9: 820p, Capacitor_SMD:C_0402_1005Metric, symbol Device:C_Small
- removed D1: PESDNC2FD5VB, easyeda2kicad:Diodes_DFN1006-2, symbol Device:D_TVS_Small
- removed D4, D92: rgb, LED_SMD:LED_Wurth_150044M155260, symbol easyeda2kicad:rgb
- removed F1: BSMD0603L-150, Fuse:Fuse_0603_1608Metric, symbol Device:Polyfuse
- removed J1: TYPE-C-31-D-06, easyeda2kicad:USB-C-SMD_TYPE-C-31-D-06, symbol Connector:USB_C_Receptacle_USB2.0_16P
- removed J2: Molex PicoBlade, Connector_Molex:Molex_PicoBlade_53261-0271_1x02-1MP_P1.25mm_Horizontal, symbol easyeda2kicad:S2B-PH-SM4-TB(LF)(SN)
- removed J3: Conn_02x06_Odd_Even, symbol Connector_Generic:Conn_02x06_Odd_Even
- removed J4: Conn_01x04_Pin, Connector_PinHeader_2.54mm:PinHeader_1x04_P2.54mm_Vertical, symbol Connector:Conn_01x04_Pin
- removed J5: 726386-2, easyeda2kicad:CONN-TH_726386-2, symbol easyeda2kicad:726386-2
- removed J6: Conn_Coaxial_Small, easyeda2kicad:IPEX-SMD_3P-L2.6-W2.6-LS3.0_ZCF-CF0001-0002IPEX, symbol Connector:Conn_Coaxial_Small
- removed J7: TF38-24S-0.5SV(830), easyeda2kicad:FPC-SMD_24P-P0.50_TF38-24S-0.5SV-830, symbol easyeda2kicad:TF38-24S-0.5SV(830)
- removed J8: FPC_12P_0.5mm, easyeda2kicad:FPC_12P_0.5mm, symbol Connector_Generic:Conn_01x12
- removed J9: FH12-12S-0.5SVA(54), easyeda2kicad:FH1212S05SVA54, symbol Connector_Generic_MountingPin:Conn_01x12_MountingPin
- removed L1: 4.7n, Inductor_SMD:L_0402_1005Metric, symbol Device:L_Small
- removed L2: 10u, Inductor_SMD:L_0603_1608Metric_Pad1.05x0.95mm_HandSolder, symbol Device:L_Small
- removed L3: 15n, Inductor_SMD:L_0402_1005Metric, symbol Device:L_Small
- removed L4: 2.2u, Inductor_SMD:L_1008_2520Metric, symbol Device:L_Small
- removed Q1: PMZB350UPE,315, Package_DFN_QFN:Diodes_DFN1006-3, symbol Device:Q_PMOS
- removed R10: 470k, Resistor_SMD:R_0402_1005Metric, symbol Device:R_Small
- removed SW89, SW91: SW_Push, easyeda2kicad:SW-SMD_2P-L3.0-W2.5-LS4.0, symbol Switch:SW_Push
- removed SW90: SW_Push, easyeda2kicad:SW-SMD_L3.9-W3.0-P4.45, symbol Switch:SW_Push
- removed TH1: 10k, symbol Device:Thermistor_NTC
- removed U1: NRF52840, nrf52840_qiaa:AQFN50P700X700X85_HS-74N, symbol nrf52840_qiaa_config5:root_0_nRF52840_QIAA_AltiumLib.DbLib
- removed U2: nPM1300-QEAA, Nordic_QFN50P500X500X90-33N:Nordic_QFN50P500X500X90-33N, symbol AltiumLib:root_0_nPM1300_QEAA_AltiumLib.DbLib
- removed U3: TPD4E05U06DQAR, Package_SON:USON-10_2.5x1.0mm_P0.5mm, symbol Power_Protection:TPD4E05U06DQA
- removed Y2: 32.768 kHz, Crystal:Crystal_SMD_3215-2Pin_3.2x1.5mm, symbol Device:Crystal_Small
- removed Yr1: 32MHz, Crystal:Crystal_SMD_2016-4Pin_2.0x1.6mm, symbol Device:Crystal_GND24_Small
Connections:
- no-connect marks 18 -> 0
Other:
- added sheet daughterboard (daughterboard.kicad_sch)
- added sheet motherboard (motherboard.kicad_sch)
- sheet matrix ports: added COL0, COL1, COL10, COL11, COL12, COL13, COL14, COL15, COL16, COL2, COL3, COL4, COL5, COL6, COL7, COL8, COL9, ROW0, ROW1, ROW2, ROW3, ROW4, ROW5; removed none
- note removed: "Backplate grounding"
- note removed: "Battery"
- note removed: "Battery terminals & Reverse polarity protection"
- note removed: "Extra pins"
- note removed: "Li-ion, Li-polymer, or LiFePO4"
- note removed: "MCU nRF52840"
- note removed: "Matrix"
- note removed: "SWD Programming & Reset"
- note removed: "TBD!!!"
- note removed: "Via to GND-layer on PVSS1"
- note removed: "ZIF Connector"
- note removed: "not req for Fxx and later"
