File: kicad/daughterboard.kicad_sch (KiCad schematic)
At the start: 9 parts, among them J1 TYPE-C-31-D-06, J8 FPC_12P_0.5mm, SW89 SW_Push, SW91 SW_Push, U3 TPD4E05U06DQAR

Commit message: update
Parts:
- D4, D92: footprint LED_SMD:LED_Wurth_150044M155260 -> easyeda2kicad:WS2812C-2020-V1
- SW89, SW91: footprint easyeda2kicad:SW-SMD_2P-L3.0-W2.5-LS4.0 -> easyeda2kicad:KEY-SMD_B3U-1000PM; LCSC Part (none) -> C231329
Changed lines of the file:
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@@
 			)
 		)
-		(property "Footprint" "LED_SMD:LED_Wurth_150044M155260"
+		(property "Footprint" "easyeda2kicad:WS2812C-2020-V1"
 			(at 162.56 81.28 0)
 			(effects
@@
 			)
 		)
-		(property "Footprint" "easyeda2kicad:SW-SMD_2P-L3.0-W2.5-LS4.0"
+		(property "Footprint" "easyeda2kicad:KEY-SMD_B3U-1000PM"
 			(at 157.48 87.63 0)
 			(effects
@@
 			)
 		)
-		(property "Datasheet" "C49234121"
+		(property "Datasheet" "www.lcsc.com/product-detail/C231329.html"
 			(at 157.48 87.63 0)
 			(effects
@@
 		)
 		(property "Description" "Push button switch, generic, two pins"
+			(at 157.48 92.71 0)
+			(effects
+				(font
+					(size 1.27 1.27)
+				)
+				(hide yes)
+			)
+		)
+		(property "LCSC Part" "C231329"
 			(at 157.48 92.71 0)
 			(effects
@@
 			)
 		)
-		(property "Footprint" "easyeda2kicad:SW-SMD_2P-L3.0-W2.5-LS4.0"
+		(property "Footprint" "easyeda2kicad:KEY-SMD_B3U-1000PM"
 			(at 157.48 97.79 0)
 			(effects
@@
 			)
 		)
-		(property "Datasheet" "C49234121"
+		(property "Datasheet" "www.lcsc.com/product-detail/C231329.html"
 			(at 157.48 97.79 0)
 			(effects
@@
 		)
 		(property "Description" "Push button switch, generic, two pins"
+			(at 157.48 102.87 0)
+			(effects
+				(font
+					(size 1.27 1.27)
+				)
+				(hide yes)
+			)
+		)
+		(property "LCSC Part" "C231329"
 			(at 157.48 102.87 0)
 			(effects
@@
 			)
 		)
-		(property "Footprint" "LED_SMD:LED_Wurth_150044M155260"
+		(property "Footprint" "easyeda2kicad:WS2812C-2020-V1"
 			(at 149.86 81.28 0)
 			(effects
