File: kicad/motherboard.kicad_sch (KiCad schematic)
At the start: 48 parts, among them J2 Molex PicoBlade, J3 Conn_02x06_Odd_Even, J4 Conn_01x04_Pin, J5 726386-2, J6 Conn_Coaxial_Small, J7 TF38-24S-0.5SV(830), J9 FH12-12S-0.5SVA(54), Q1 PMZB350UPE,315, SW90 SW_Push, U1 NRF52840, U2 nPM1300-QEAA, Y1 32MHz, Y2 32.768 kHz

Commit message: update
Parts:
- SW90: footprint easyeda2kicad:SW-SMD_L3.9-W3.0-P4.45 -> easyeda2kicad:SW-SMD_2P-L3.0-W2.5-LS4.0; LCSC Part C720477 -> C49234121
Changed lines of the file:
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@@
 			)
 		)
-		(property "Footprint" "easyeda2kicad:SW-SMD_L3.9-W3.0-P4.45"
+		(property "Footprint" "easyeda2kicad:SW-SMD_2P-L3.0-W2.5-LS4.0"
 			(at 130.81 236.22 0)
 			(effects
@@
 			)
 		)
-		(property "Datasheet" "https://www.lcsc.com/product-detail/C720477.html"
+		(property "Datasheet" "C49234121"
 			(at 130.81 236.22 0)
 			(effects
@@
 			)
 		)
-		(property "LCSC Part" "C720477"
+		(property "LCSC Part" "C49234121"
 			(at 130.81 241.3 0)
 			(effects
-				(font
-					(size 1.27 1.27)
-				)
-				(hide yes)
-			)
-		)
-		(property "Sim.Pin" ""
-			(at 130.81 241.3 0)
-			(effects

Commit message: update
Parts:
- removed J4: Conn_01x04_Pin, Connector_PinHeader_2.54mm:PinHeader_1x04_P2.54mm_Vertical, symbol Connector:Conn_01x04_Pin
- added J10: TC2030, Connector:Tag-Connect_TC2030-IDC-NL_2x03_P1.27mm_Vertical, symbol Connector:TC2030
Connections:
- net GND: now also J10.3, J10.5
- net SWCLK: now also J10.4
- net SWDIO: now also J10.2
- net VDD_NRF: now also J10.1
- new net SWO: J10.6

Commit message: update
Parts:
- removed J7: TF38-24S-0.5SV(830), easyeda2kicad:FPC-SMD_24P-P0.50_TF38-24S-0.5SV-830, symbol easyeda2kicad:TF38-24S-0.5SV(830)
- added J4: AFB10-S18LCA-00, easyeda2kicad:FPC-SMD_18P-P1.00_AFB10-S18LCA-00, symbol Connector_Generic_MountingPin:Conn_01x18_MountingPin
- added J7: AFB10-S06LCA-00, easyeda2kicad:FPC-SMD_6P-P1.00_AFB10-S6LCA-00, symbol Connector_Generic_MountingPin:Conn_01x06_MountingPin
- J9: value FH12-12S-0.5SVA(54) -> AFC11-S12ICA-00; footprint easyeda2kicad:FH1212S05SVA54 -> easyeda2kicad:CONN-SMD-12P_AFC11-S12ICA-00; LCSC Part C3168197 -> C262499
- Q1: footprint Package_DFN_QFN:Diodes_DFN1006-3 -> easyeda2kicad:DFN1006-3
- SW90: footprint easyeda2kicad:SW-SMD_2P-L3.0-W2.5-LS4.0 -> easyeda2kicad:KEY-SMD_B3U-1000PM; LCSC Part C49234121 -> C231329
- Y1: footprint Crystal:Crystal_SMD_2016-4Pin_2.0x1.6mm -> easyeda2kicad:Crystal_SMD_2016-4Pin_2.0x1.6mm
- Y2: footprint Crystal:Crystal_SMD_3215-2Pin_3.2x1.5mm -> easyeda2kicad:Crystal_SMD_3215-2Pin
Other:
- note added: "FPC Connector"
- note removed: "ZIF Connector"
- moved on the sheet: Y1
