File: hardware/controller/controller.kicad_pcb (KiCad board)
At the start: 4 copper layers, 75 x 50 mm, 55 parts, among them J1 TYPE-C-31-D-06, J10 TC2030, J2 Molex PicoBlade, J4 AFB10-S18LCA-00, J5 726386-2, J6 Conn_Coaxial_Small, J7 AFB10-S06LCA-00, J8 FPC_12P_0.5mm, J9 AFC11-S12ICA-00, Q1 PMZB350UPE,315, SW89 SW_Push, SW90 SW_Push, SW91 SW_Push, U1 NRF52840, U2 nPM1300-QEAA, U3 TPD4E05U06DQAR, Y1 32MHz, Y2 32.768 kHz

Commit message: feat(controller): update PCB from schematic, footprint cleanup, DRC in check script
- PCB updated from the split schematic: new parts placed (C19, C35, D2, J3,
  L5, NT1, Q2, R1/R2, R11/R12, SW1, TP1), old ones removed (D4, D92,
  SW89-91, old Q1, C10), footprints replaced (J2 JST PH, J8/J9 1x10 1.0 mm,
  F1 1210, D1 SOD-123F).
- Footprint fixes: J1 shield pads, pad rounding, silkscreen; standard
  footprints with local changes copied to ibm_bs.pretty (JST PH, headers,
  SOT-23, test pad).
- tools/kicad-check.sh: PCB DRC with schematic parity.
Parts:
- removed C10: NC, Capacitor_SMD:C_0402_1005Metric
- removed D4, D92: rgb, easyeda2kicad:WS2812C-2020-V1
- removed Q1: PMZB350UPE,315, easyeda2kicad:DFN1006-3
- removed SW89, SW90, SW91: SW_Push, easyeda2kicad:KEY-SMD_B3U-1000PM
- added C19: 100n, Capacitor_SMD:C_0402_1005Metric, F.Cu at (86.2, 107.5)
- added C35: 100n, Capacitor_SMD:C_0402_1005Metric, F.Cu at (86.2, 109.5)
- added D2: WS2812B-2020-V6, easyeda2kicad:LED-SMD_4P-L2.2-W2.0-P1.00_WS2815C-2020-4P, F.Cu at (89.4, 108.1)
- added J3: PinHeader_2x03_P1.27mm, ibm_bs:PinHeader_2x03_P1.27mm_Vertical_SMD, F.Cu at (64.5, 109.0)
- added L5: 2.2n, Inductor_SMD:L_0402_1005Metric, F.Cu at (83.3, 103.1)
- added NT1: NetTie, NetTie:NetTie-2_THT_Pad0.3mm, F.Cu at (85.5, 111.3)
- added Q2: AO3401A, ibm_bs:SOT-23, F.Cu at (87.2, 104.3)
- added R1: 0, Resistor_SMD:R_0402_1005Metric, F.Cu at (83.3, 105.1)
- added R11: 4.7k, Resistor_SMD:R_0402_1005Metric, F.Cu at (83.3, 109.0)
- added R12: 4.7k, Resistor_SMD:R_0402_1005Metric, F.Cu at (83.3, 111.0)
- added R2: 0, Resistor_SMD:R_0402_1005Metric, F.Cu at (83.3, 107.0)
- added SW1: SW_Push, easyeda2kicad:SW-SMD_4P-L5.1-W5.1-P3.70-LS6.5-TL_H1.5, F.Cu at (74.5, 108.5)
- added TP1: TestPoint, ibm_bs:TestPoint_Pad, F.Cu at (88.5, 110.5)
- C16: footprint Capacitor_SMD:C_0402_1005Metric -> Capacitor_SMD:C_0603_1608Metric
- C3: value 0.8p -> 1p
- C4: value 0.5p -> 1.2p
- C9: value 820p -> DNP
- D1: value PESDNC2FD5VB -> SMF20A; footprint easyeda2kicad:Diodes_DFN1006-2 -> Diode_SMD:D_SOD-123F
- F1: value BSMD0603L-150 -> SMD1210-110-24V; footprint Fuse:Fuse_0603_1608Metric -> Fuse:Fuse_1210_3225Metric
- J2: value Molex PicoBlade -> JST-PH-1x02_P2.00mm; footprint Connector_Molex:Molex_PicoBlade_53261-0271_1x02-1MP_P1.25mm_Horizontal -> ibm_bs:JST_PH_S2B-PH-SM4-TB_1x02-1MP_P2.00mm_Horizontal
- J5: value 726386-2 -> Backplate GND
- J6: value Conn_Coaxial_Small -> ~; footprint easyeda2kicad:IPEX-SMD_3P-L2.6-W2.6-LS3.0_ZCF-CF0001-0002IPEX -> easyeda2kicad:IPEX-SMD_4P-L2.6-W2.6-LS3.0_GT-RF1125A-01G
- J8: value FPC_12P_0.5mm -> Header_1x10_P1.00mm; footprint easyeda2kicad:FPC_12P_0.5mm -> ibm_bs:PinHeader_1x10_P1.00mm_Vertical_SMD_Pin1Left
- J9: value AFC11-S12ICA-00 -> Header_1x10_P1.00mm; footprint easyeda2kicad:CONN-SMD-12P_AFC11-S12ICA-00 -> ibm_bs:PinHeader_1x10_P1.00mm_Vertical
- R10: footprint Resistor_SMD:R_0402_1005Metric -> Resistor_SMD:R_0603_1608Metric
- U1: value NRF52840 -> nRF52840-QIAA
- moved J9 7.55 mm to (62.0, 73.5), turned to 90 degrees
- moved F1 6.34 mm to (103.3, 96.9)
- moved J8 5.66 mm to (89.5, 91.0), turned to 180 degrees
- moved D1 1.79 mm to (95.8, 98.4)
Connections:
- net /motherboard/DEC4 renamed Net-(U1B-DEC4)
- net /motherboard/SWCLK renamed /MCU IO/SWCLK
- net /motherboard/SWDIO renamed /MCU IO/SWDIO
- net Net-(U2-LSOUT1/VOUTLDO1) renamed VLED
- C1 pad 1: GND -> Net-(U1C-XC2)
- C1 pad 2: Net-(U1-XC1) -> GND
- C17 pad 1: GND -> Net-(U1C-P0.01/XL2)
- C17 pad 2: Net-(U1-P0.00/XL1) -> GND
- C18 pad 2: Net-(U1-P0.01/XL2) -> Net-(U1C-P0.00/XL1)
- C2 pad 2: Net-(U1-XC2) -> Net-(U1C-XC1)
- C29 pad 2: PVSS1 -> PVSS2
- C30 pad 2: PVSS1 -> PVSS2
- C4 pad 1: /motherboard/ANTENNA -> Net-(C4-Pad1)
- D1 pad 1: GND -> DB_VBUS
- D1 pad 2: VBUS -> DB_GND
- F1 pad 2: VBUS -> DB_VBUS
- J1 pad A1: GND -> DB_GND
- J1 pad A12: GND -> DB_GND
- J1 pad A5: /daughterboard/CC1 -> /Daughterboard/DB_CC1
- J1 pad A6: D+ -> /Daughterboard/DB_D+
- J1 pad A7: D- -> /Daughterboard/DB_D-
- J1 pad B1: GND -> DB_GND
- J1 pad B12: GND -> DB_GND
- J1 pad B5: /daughterboard/CC2 -> /Daughterboard/DB_CC2
- J1 pad B6: D+ -> /Daughterboard/DB_D+
- J1 pad B7: D- -> /Daughterboard/DB_D-
- J10 pad 3: GND -> /MCU IO/RESET
- J10 pad 6: /motherboard/SWO -> /MCU IO/SWO
- J2 pad MP: (no net) -> GND
- J4 pad 1: unconnected-(J4-Pin_1-Pad1) -> /MCU IO/COL0
- J4 pad 10: unconnected-(J4-Pin_10-Pad10) -> /MCU IO/COL9
- J4 pad 11: unconnected-(J4-Pin_11-Pad11) -> /MCU IO/COL10
- J4 pad 12: unconnected-(J4-Pin_12-Pad12) -> /MCU IO/COL11
- J4 pad 13: unconnected-(J4-Pin_13-Pad13) -> /MCU IO/COL12
- J4 pad 14: unconnected-(J4-Pin_14-Pad14) -> /MCU IO/COL13
- J4 pad 15: unconnected-(J4-Pin_15-Pad15) -> /MCU IO/COL14
- J4 pad 16: unconnected-(J4-Pin_16-Pad16) -> /MCU IO/COL15
- J4 pad 17: unconnected-(J4-Pin_17-Pad17) -> /MCU IO/COL16
- J4 pad 18: unconnected-(J4-Pin_18-Pad18) -> GND
- J4 pad 2: unconnected-(J4-Pin_2-Pad2) -> /MCU IO/COL1
- J4 pad 3: unconnected-(J4-Pin_3-Pad3) -> /MCU IO/COL2
- J4 pad 4: unconnected-(J4-Pin_4-Pad4) -> /MCU IO/COL3
- J4 pad 5: unconnected-(J4-Pin_5-Pad5) -> /MCU IO/COL4
- J4 pad 6: unconnected-(J4-Pin_6-Pad6) -> /MCU IO/COL5
- J4 pad 7: unconnected-(J4-Pin_7-Pad7) -> /MCU IO/COL6
- J4 pad 8: unconnected-(J4-Pin_8-Pad8) -> /MCU IO/COL7
- J4 pad 9: unconnected-(J4-Pin_9-Pad9) -> /MCU IO/COL8
- J6 pad 1: /motherboard/ANTENNA -> Net-(J6-In)
- J7 pad 1: unconnected-(J7-Pin_1-Pad1) -> /MCU IO/ROW0
- J7 pad 2: unconnected-(J7-Pin_2-Pad2) -> /MCU IO/ROW1
- J7 pad 3: unconnected-(J7-Pin_3-Pad3) -> /MCU IO/ROW2
- J7 pad 4: unconnected-(J7-Pin_4-Pad4) -> /MCU IO/ROW3
- J7 pad 5: unconnected-(J7-Pin_5-Pad5) -> /MCU IO/ROW4
- J7 pad 6: unconnected-(J7-Pin_6-Pad6) -> /MCU IO/ROW5
- J8 pad 1: VBUS -> DB_VBUS
- J8 pad 10: /daughterboard/LED_DATA -> DB_GND
- J8 pad 2: VBUS -> DB_VBUS
- J8 pad 3: /daughterboard/BT_PAIR -> /Daughterboard/DB_CC1
- J8 pad 4: /daughterboard/CC1 -> DB_GND
- J8 pad 5: GND -> /Daughterboard/DB_D+
- J8 pad 6: D+ -> /Daughterboard/DB_D-
- J8 pad 7: D- -> DB_GND
- J8 pad 8: GND -> /Daughterboard/DB_CC2
- J8 pad 9: /daughterboard/CC2 -> DB_GND
- J9 pad 10: /daughterboard/LED_DATA -> GND
- J9 pad 3: /daughterboard/BT_PAIR -> /Power/CC1
- J9 pad 4: /daughterboard/CC1 -> GND
- J9 pad 5: GND -> D+
- J9 pad 6: D+ -> D-
- J9 pad 7: D- -> GND
- J9 pad 8: GND -> /Power/CC2
- J9 pad 9: /daughterboard/CC2 -> GND
- L1 pad 2: /motherboard/ANTENNA -> Net-(C4-Pad1)
- L4 pad 1: VDD_NRF -> Net-(U2-SW2)
- L4 pad 2: Net-(U2-SW1) -> VDD_NRF
- R10 pad 1: Net-(U2-VSET1) -> Net-(U2-VSET2)
- U1 pad A10: unconnected-(U1-P0.29/AIN5-PadA10) -> /MCU IO/COL3
- U1 pad A12: unconnected-(U1-P0.02/AIN0-PadA12) -> /MCU IO/COL0
- U1 pad A14: unconnected-(U1-P1.15-PadA14) -> /MCU IO/COL11
- U1 pad A16: unconnected-(U1-P1.13-PadA16) -> /MCU IO/COL9
- U1 pad A18: Net-(U1-DEC2) -> unconnected-(U1B-DEC2-PadA18)
- U1 pad A20: unconnected-(U1-P1.10-PadA20) -> /MCU IO/COL6
- U1 pad A23: Net-(U1-XC2) -> Net-(U1C-XC2)
- U1 pad A8: unconnected-(U1-P0.31/AIN7-PadA8) -> /MCU IO/COL5
- U1 pad AC13: unconnected-(U1-P0.18/RESET-PadAC13) -> /MCU IO/RESET
- U1 pad AC15: unconnected-(U1-P0.19-PadAC15) -> /MCU IO/EXT_INT
- U1 pad AC9: unconnected-(U1-P0.14-PadAC9) -> SCL
- U1 pad AD10: unconnected-(U1-P0.15-PadAD10) -> /MCU IO/RGB_DIN
- U1 pad AD22: unconnected-(U1-P1.00-PadAD22) -> /MCU IO/SWO
- U1 pad AD8: unconnected-(U1-P0.13-PadAD8) -> SDA
- U1 pad B11: unconnected-(U1-P0.28/AIN4-PadB11) -> /MCU IO/COL2
- U1 pad B13: unconnected-(U1-P0.03/AIN1-PadB13) -> /MCU IO/COL1
- U1 pad B15: unconnected-(U1-P1.14-PadB15) -> /MCU IO/COL10
- U1 pad B17: unconnected-(U1-P1.12-PadB17) -> /MCU IO/COL8
- U1 pad B19: unconnected-(U1-P1.11-PadB19) -> /MCU IO/COL7
- U1 pad B24: Net-(U1-XC1) -> Net-(U1C-XC1)
- U1 pad B9: unconnected-(U1-P0.30/AIN6-PadB9) -> /MCU IO/COL4
- U1 pad D2: Net-(U1-P0.00/XL1) -> Net-(U1C-P0.00/XL1)
- U1 pad F2: Net-(U1-P0.01/XL2) -> Net-(U1C-P0.01/XL2)
- U1 pad G1: unconnected-(U1-P0.26-PadG1) -> /MCU IO/COL13
- U1 pad H2: unconnected-(U1-P0.27-PadH2) -> /MCU IO/COL14
- U1 pad J1: unconnected-(U1-P0.04/AIN2-PadJ1) -> /MCU IO/ROW0
- U1 pad K2: unconnected-(U1-P0.05/AIN3-PadK2) -> /MCU IO/ROW1
- U1 pad L1: unconnected-(U1-P0.06-PadL1) -> /MCU IO/ROW2
- U1 pad M2: unconnected-(U1-P0.07-PadM2) -> /MCU IO/ROW3
- U1 pad N1: unconnected-(U1-P0.08-PadN1) -> /MCU IO/ROW4
- U1 pad P2: unconnected-(U1-P1.08-PadP2) -> /MCU IO/COL15
- U1 pad R1: unconnected-(U1-P1.09-PadR1) -> /MCU IO/COL16
- U1 pad T2: unconnected-(U1-P0.11-PadT2) -> /MCU IO/ROW5
- U1 pad U1: unconnected-(U1-P0.12-PadU1) -> /MCU IO/COL12
- U1 pad W24: unconnected-(U1-P1.02-PadW24) -> LED_EN
- U1 pad Y23: unconnected-(U1-P1.01-PadY23) -> PMIC_INT
- U2 pad 1: VDD_NRF -> VSYS
- U2 pad 12: unconnected-(U2-VDDIO-Pad12) -> VDD_NRF
- U2 pad 13: /motherboard/SDA -> SDA
- U2 pad 14: /motherboard/SCL -> SCL
- U2 pad 15: /daughterboard/SHPHLD -> /Power/SHPHLD
- U2 pad 16: GND -> Net-(U2-VSET2)
- U2 pad 17: Net-(U2-VSET1) -> GND
- U2 pad 18: Net-(U2-NTC) -> GND
- U2 pad 2: PVSS1 -> GND
- U2 pad 23: /daughterboard/CC1 -> /Power/CC1
- U2 pad 24: /daughterboard/CC2 -> /Power/CC2
- U2 pad 28: VDD_NRF -> VSYS
- U2 pad 3: Net-(U2-SW1) -> unconnected-(U2-SW1-Pad3)
- U2 pad 32: VSYS -> VDD_NRF
- U2 pad 5: unconnected-(U2-SW2-Pad5) -> Net-(U2-SW2)
- U2 pad 6: GND -> PVSS2
- U2 pad 7: unconnected-(U2-GPIO0-Pad7) -> PMIC_INT
- U2 pad 8: unconnected-(U2-GPIO1-Pad8) -> LED_EN
- U3 pad 1: /daughterboard/CC1 -> /Daughterboard/DB_CC1
- U3 pad 10: /daughterboard/CC1 -> /Daughterboard/DB_CC1
- U3 pad 2: D+ -> /Daughterboard/DB_D+
- U3 pad 3: GND -> DB_GND
- U3 pad 4: D- -> /Daughterboard/DB_D-
- U3 pad 5: /daughterboard/CC2 -> /Daughterboard/DB_CC2
- U3 pad 6: /daughterboard/CC2 -> /Daughterboard/DB_CC2
- U3 pad 7: D- -> /Daughterboard/DB_D-
- U3 pad 8: GND -> DB_GND
- U3 pad 9: D+ -> /Daughterboard/DB_D+
- Y1 pad 1: Net-(U1-XC2) -> Net-(U1C-XC1)
- Y1 pad 3: Net-(U1-XC1) -> Net-(U1C-XC2)
- Y2 pad 1: Net-(U1-P0.01/XL2) -> Net-(U1C-P0.00/XL1)
- Y2 pad 2: Net-(U1-P0.00/XL1) -> Net-(U1C-P0.01/XL2)
Routing:
- net (no net): track 0.00 -> 32.1 mm, vias 0 -> 4
- net D-: track 12.8 -> 0.00 mm, vias 2 -> 0
- net /Daughterboard/DB_D-: track 0.00 -> 12.8 mm, vias 0 -> 2
- net D+: track 12.8 -> 0.00 mm, vias 2 -> 0
- net /Daughterboard/DB_D+: track 0.00 -> 12.8 mm, vias 0 -> 2
- net /daughterboard/CC2: track 10.6 -> 0.00 mm, vias 3 -> 0
- net GND: track 43.4 -> 53.7 mm, vias 35 -> 28
- net /daughterboard/SHPHLD: track 10.3 -> 0.00 mm, vias 3 -> 0
- net DB_GND: track 0.00 -> 10.1 mm, vias 0 -> 6
- net /daughterboard/BT_PAIR: track 9.85 -> 0.00 mm, vias 2 -> 0
- net /daughterboard/CC1: track 8.22 -> 0.00 mm, vias 1 -> 0
- net /Daughterboard/DB_CC2: track 0.00 -> 7.43 mm, vias 0 -> 2
- net Net-(U1-P0.00/XL1): track 7.14 -> 0.00 mm
- net VBUS: track 6.61 -> 0.00 mm
- net Net-(U1-XC1): track 6.18 -> 0.00 mm
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- added copper zone on F.Cu, net GND
- removed copper zone on F.Cu, net PVSS1
