File: hardware/controller/io.kicad_sch (KiCad schematic)
At the start: 13 parts, among them J10 TC2030, J3 PinHeader_2x03_P1.27mm, J4 AFB10-S18LCA-00, J5 Backplate GND, J7 AFB10-S06LCA-00, SW1 SW_Push, U1 nRF52840-QIAA

Commit message: feat(controller): update PCB from schematic, footprint cleanup, DRC in check script
- PCB updated from the split schematic: new parts placed (C19, C35, D2, J3,
  L5, NT1, Q2, R1/R2, R11/R12, SW1, TP1), old ones removed (D4, D92,
  SW89-91, old Q1, C10), footprints replaced (J2 JST PH, J8/J9 1x10 1.0 mm,
  F1 1210, D1 SOD-123F).
- Footprint fixes: J1 shield pads, pad rounding, silkscreen; standard
  footprints with local changes copied to ibm_bs.pretty (JST PH, headers,
  SOT-23, test pad).
- tools/kicad-check.sh: PCB DRC with schematic parity.
Parts:
- J3: footprint Connector_PinHeader_1.27mm:PinHeader_2x03_P1.27mm_Vertical_SMD -> ibm_bs:PinHeader_2x03_P1.27mm_Vertical_SMD
Changed lines of the file:
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@@
 			)
 		)
-		(property "Footprint" "Connector_PinHeader_1.27mm:PinHeader_2x03_P1.27mm_Vertical_SMD"
+		(property "Footprint" "ibm_bs:PinHeader_2x03_P1.27mm_Vertical_SMD"
 			(at 91.44 180.34 0)
 			(hide yes)
