File: hardware/controller/power.kicad_sch (KiCad schematic)
At the start: 16 parts, among them J2 JST-PH-1x02_P2.00mm, J9 Header_1x10_P1.00mm, Q2 AO3401A, U2 nPM1300-QEAA

Commit message: feat(controller): update PCB from schematic, footprint cleanup, DRC in check script
- PCB updated from the split schematic: new parts placed (C19, C35, D2, J3,
  L5, NT1, Q2, R1/R2, R11/R12, SW1, TP1), old ones removed (D4, D92,
  SW89-91, old Q1, C10), footprints replaced (J2 JST PH, J8/J9 1x10 1.0 mm,
  F1 1210, D1 SOD-123F).
- Footprint fixes: J1 shield pads, pad rounding, silkscreen; standard
  footprints with local changes copied to ibm_bs.pretty (JST PH, headers,
  SOT-23, test pad).
- tools/kicad-check.sh: PCB DRC with schematic parity.
Parts:
- J2: footprint Connector_JST:JST_PH_S2B-PH-SM4-TB_1x02-1MP_P2.00mm_Horizontal -> ibm_bs:JST_PH_S2B-PH-SM4-TB_1x02-1MP_P2.00mm_Horizontal
- J9: footprint Connector_PinHeader_1.00mm:PinHeader_1x10_P1.00mm_Vertical -> ibm_bs:PinHeader_1x10_P1.00mm_Vertical
- Q2: footprint Package_TO_SOT_SMD:SOT-23 -> ibm_bs:SOT-23
- TP1: footprint TestPoint:TestPoint_Pad_D1.0mm -> ibm_bs:TestPoint_Pad
Changed lines of the file:
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@@
 			)
 		)
-		(property "Footprint" "Connector_JST:JST_PH_S2B-PH-SM4-TB_1x02-1MP_P2.00mm_Horizontal"
+		(property "Footprint" "ibm_bs:JST_PH_S2B-PH-SM4-TB_1x02-1MP_P2.00mm_Horizontal"
 			(at 83.82 64.77 0)
 			(hide yes)
@@
 			)
 		)
-		(property "Footprint" "Package_TO_SOT_SMD:SOT-23"
+		(property "Footprint" "ibm_bs:SOT-23"
 			(at 110.49 64.77 0)
 			(hide yes)
@@
 			)
 		)
-		(property "Footprint" "TestPoint:TestPoint_Pad_D1.0mm"
+		(property "Footprint" "ibm_bs:TestPoint_Pad"
 			(at 133.35 82.55 0)
 			(hide yes)
@@
 			)
 		)
-		(property "Footprint" "Connector_PinHeader_1.00mm:PinHeader_1x10_P1.00mm_Vertical"
+		(property "Footprint" "ibm_bs:PinHeader_1x10_P1.00mm_Vertical"
 			(at 45.72 54.61 0)
 			(hide yes)
